File: hardware/IVC-k30/CPU.kicad_sch (KiCad schematic)
At the start: 19 parts, among them SW1 ~{RESET}, U1 MC68030FE, U2 74HC14, U3 74HC05, Y1 Crystal

Commit message: Updated k30 CPU card
Parts:
- renumbered C4 to C2, C5 to C3
Connections:
- net A0 renamed LA0
- net A1 renamed LA1
- net A10 renamed LA10
- net A11 renamed LA11
- net A12 renamed LA12
- net A13 renamed LA13
- net A14 renamed LA14
- net A15 renamed LA15
- net A16 renamed LA16
- net A17 renamed LA17
- net A18 renamed LA18
- net A19 renamed LA19
- net A2 renamed LA2
- net A20 renamed LA20
- net A21 renamed LA21
- net A22 renamed LA22
- net A23 renamed LA23
- net A24 renamed LA24
- net A25 renamed LA25
- net A26 renamed LA26
- net A27 renamed LA27
- net A28 renamed LA28
- net A29 renamed LA29
- net A3 renamed LA3
- net A30 renamed LA30
- net A31 renamed LA31
- net A4 renamed LA4
- net A5 renamed LA5
- net A6 renamed LA6
- net A7 renamed LA7
- net A8 renamed LA8
- net A9 renamed LA9
- net D0 renamed LD0
- net D1 renamed LD1
- net D10 renamed LD10
- net D11 renamed LD11
- net D12 renamed LD12
- net D13 renamed LD13
- net D14 renamed LD14
- net D15 renamed LD15
- net D16 renamed LD16
- net D17 renamed LD17
- net D18 renamed LD18
- net D19 renamed LD19
- net D2 renamed LD2
- net D20 renamed LD20
- net D21 renamed LD21
- net D22 renamed LD22
- net D23 renamed LD23
- net D24 renamed LD24
- net D25 renamed LD25
- net D26 renamed LD26
- net D27 renamed LD27
- net D28 renamed LD28
- net D29 renamed LD29
- net D3 renamed LD3
- net D30 renamed LD30
- net D31 renamed LD31
- net D4 renamed LD4
- net D5 renamed LD5
- net D6 renamed LD6
- net D7 renamed LD7
- net D8 renamed LD8
- net D9 renamed LD9
Other:
- moved on the sheet: C1, C2, C3, D1, R1, R2, R3, R4, RN1, RN2, SW1, U2A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
