File: hardware/IVC-k30/IO.kicad_sch (KiCad schematic)
At the start: 26 parts, among them J1 CompactFlash, J2 Serial1, J3 Serial2, SW3 IP2, SW4 IP3, U13 MC68681, U7 74HC32, Y2 Crystal

Commit message: Updated k30 CPU card
Parts:
- renumbered C2 to C4, C3 to C5, J1 to J2, J2 to J3, J3 to J4, JP2 to JP1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
