File: hardware/IVC-k30/Memory.kicad_sch (KiCad schematic)
At the start: 3 parts, among them U14 AS6C8016, U15 AS6C8016, U16 AM29F040

Commit message: Updated k30 CPU card
Parts:
- renumbered U14 to U5, U15 to U6, U16 to U7
Changed lines of the file:
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@@
   (symbol (lib_id "Computie_Memory:AS6C8016") (at 76.2 58.42 0) (unit 1)
     (in_bom yes) (on_board yes) (dnp no)
-    (property "Reference" "U14" (at 76.2 25.8826 0)
+    (property "Reference" "U5" (at 76.2 25.8826 0)
       (effects (font (size 1.27 1.27)))
     )
@@
       (project "IVC-k30"
         (path "/dd13a6b9-cb24-4a73-96ce-c29930072fba/69e17b68-518f-4a96-bc5f-1d2df7d01a56"
+          (reference "U5") (unit 1)
+        )
+      )
+      (project "k30-SBC"
+        (path "/fc911c32-ec9d-4dc3-a64d-23ac8e8e7030/00000000-0000-0000-0000-0000613dffc0"
           (reference "U14") (unit 1)
         )
       )
-      (project "k30-SBC"
-        (path "/fc911c32-ec9d-4dc3-a64d-23ac8e8e7030/00000000-0000-0000-0000-0000613dffc0"
-          (reference "U14") (unit 1)
-        )
-      )
     )
   )
   (symbol (lib_id "Computie_Memory:AS6C8016") (at 76.2 138.43 0) (unit 1)
     (in_bom yes) (on_board yes) (dnp no)
-    (property "Reference" "U15" (at 76.2 105.8926 0)
+    (property "Reference" "U6" (at 76.2 105.8926 0)
       (effects (font (size 1.27 1.27)))
     )
@@
       (project "IVC-k30"
         (path "/dd13a6b9-cb24-4a73-96ce-c29930072fba/69e17b68-518f-4a96-bc5f-1d2df7d01a56"
+          (reference "U6") (unit 1)
+        )
+      )
+      (project "k30-SBC"
+        (path "/fc911c32-ec9d-4dc3-a64d-23ac8e8e7030/00000000-0000-0000-0000-0000613dffc0"
           (reference "U15") (unit 1)
         )
       )
-      (project "k30-SBC"
-        (path "/fc911c32-ec9d-4dc3-a64d-23ac8e8e7030/00000000-0000-0000-0000-0000613dffc0"
-          (reference "U15") (unit 1)
-        )
-      )
     )
   )
   (symbol (lib_id "power:+5V") (at 85.09 30.48 0) (unit 1)
     (in_bom yes) (on_board yes) (dnp no)
-    (property "Reference" "#PWR034" (at 85.09 34.29 0)
+    (property "Reference" "#PWR014" (at 85.09 34.29 0)
       (effects (font (size 1.27 1.27)) hide)
     )
@@
       (project "IVC-k30"
         (path "/dd13a6b9-cb24-4a73-96ce-c29930072fba/69e17b68-518f-4a96-bc5f-1d2df7d01a56"
+          (reference "#PWR014") (unit 1)
+        )
+      )
+      (project "k30-SBC"
+        (path "/fc911c32-ec9d-4dc3-a64d-23ac8e8e7030/00000000-0000-0000-0000-0000613dffc0"
           (reference "#PWR034") (unit 1)
         )
       )
-      (project "k30-SBC"
-        (path "/fc911c32-ec9d-4dc3-a64d-23ac8e8e7030/00000000-0000-0000-0000-0000613dffc0"
-          (reference "#PWR034") (unit 1)
-        )
-      )
     )
   )
   (symbol (lib_id "power:GND") (at 76.2 92.71 0) (unit 1)
     (in_bom yes) (on_board yes) (dnp no)
-    (property "Reference" "#PWR032" (at 76.2 99.06 0)
+    (property "Reference" "#PWR012" (at 76.2 99.06 0)
       (effects (font (size 1.27 1.27)) hide)
     )
@@
       (project "IVC-k30"
         (path "/dd13a6b9-cb24-4a73-96ce-c29930072fba/69e17b68-518f-4a96-bc5f-1d2df7d01a56"
+          (reference "#PWR012") (unit 1)
+        )
+      )
+      (project "k30-SBC"
+        (path "/fc911c32-ec9d-4dc3-a64d-23ac8e8e7030/00000000-0000-0000-0000-0000613dffc0"
           (reference "#PWR032") (unit 1)
         )
       )
-      (project "k30-SBC"
-        (path "/fc911c32-ec9d-4dc3-a64d-23ac8e8e7030/00000000-0000-0000-0000-0000613dffc0"
-          (reference "#PWR032") (unit 1)
-        )
-      )
     )
   )
   (symbol (lib_id "power:GND") (at 76.2 172.72 0) (unit 1)
     (in_bom yes) (on_board yes) (dnp no)
-    (property "Reference" "#PWR033" (at 76.2 179.07 0)
+    (property "Reference" "#PWR013" (at 76.2 179.07 0)
       (effects (font (size 1.27 1.27)) hide)
     )
@@
       (project "IVC-k30"
         (path "/dd13a6b9-cb24-4a73-96ce-c29930072fba/69e17b68-518f-4a96-bc5f-1d2df7d01a56"
+          (reference "#PWR013") (unit 1)
+        )
+      )
+      (project "k30-SBC"
+        (path "/fc911c32-ec9d-4dc3-a64d-23ac8e8e7030/00000000-0000-0000-0000-0000613dffc0"
           (reference "#PWR033") (unit 1)
         )
       )
-      (project "k30-SBC"
-        (path "/fc911c32-ec9d-4dc3-a64d-23ac8e8e7030/00000000-0000-0000-0000-0000613dffc0"
-          (reference "#PWR033") (unit 1)
-        )
-      )
     )
   )
   (symbol (lib_id "power:+5V") (at 85.09 110.49 0) (unit 1)
     (in_bom yes) (on_board yes) (dnp no)
-    (property "Reference" "#PWR035" (at 85.09 114.3 0)
+    (property "Reference" "#PWR015" (at 85.09 114.3 0)
       (effects (font (size 1.27 1.27)) hide)
     )
@@
       (project "IVC-k30"
         (path "/dd13a6b9-cb24-4a73-96ce-c29930072fba/69e17b68-518f-4a96-bc5f-1d2df7d01a56"
+          (reference "#PWR015") (unit 1)
+        )
+      )
+      (project "k30-SBC"
+        (path "/fc911c32-ec9d-4dc3-a64d-23ac8e8e7030/00000000-0000-0000-0000-0000613dffc0"
           (reference "#PWR035") (unit 1)
         )
       )
-      (project "k30-SBC"
-        (path "/fc911c32-ec9d-4dc3-a64d-23ac8e8e7030/00000000-0000-0000-0000-0000613dffc0"
-          (reference "#PWR035") (unit 1)
-        )
-      )
     )
   )
   (symbol (lib_id "Computie_Memory:AM29F040") (at 176.53 55.88 0) (unit 1)
     (in_bom yes) (on_board yes) (dnp no)
-    (property "Reference" "U16" (at 176.53 25.8826 0)
+    (property "Reference" "U7" (at 176.53 25.8826 0)
       (effects (font (size 1.27 1.27)))
     )
@@
       (project "IVC-k30"
         (path "/dd13a6b9-cb24-4a73-96ce-c29930072fba/69e17b68-518f-4a96-bc5f-1d2df7d01a56"
+          (reference "U7") (unit 1)
+        )
+      )
+      (project "k30-SBC"
+        (path "/fc911c32-ec9d-4dc3-a64d-23ac8e8e7030/00000000-0000-0000-0000-0000613dffc0"
           (reference "U16") (unit 1)
         )
       )
-      (project "k30-SBC"
-        (path "/fc911c32-ec9d-4dc3-a64d-23ac8e8e7030/00000000-0000-0000-0000-0000613dffc0"
-          (reference "U16") (unit 1)
-        )
-      )
     )
   )
   (symbol (lib_id "power:+5V") (at 185.42 30.48 0) (unit 1)
     (in_bom yes) (on_board yes) (dnp no)
-    (property "Reference" "#PWR037" (at 185.42 34.29 0)
+    (property "Reference" "#PWR017" (at 185.42 34.29 0)
       (effects (font (size 1.27 1.27)) hide)
     )
@@
       (project "IVC-k30"
         (path "/dd13a6b9-cb24-4a73-96ce-c29930072fba/69e17b68-518f-4a96-bc5f-1d2df7d01a56"
+          (reference "#PWR017") (unit 1)
+        )
+      )
+      (project "k30-SBC"
+        (path "/fc911c32-ec9d-4dc3-a64d-23ac8e8e7030/00000000-0000-0000-0000-0000613dffc0"
           (reference "#PWR037") (unit 1)
         )
       )
-      (project "k30-SBC"
-        (path "/fc911c32-ec9d-4dc3-a64d-23ac8e8e7030/00000000-0000-0000-0000-0000613dffc0"
-          (reference "#PWR037") (unit 1)
-        )
-      )
     )
   )
   (symbol (lib_id "power:GND") (at 176.53 86.36 0) (unit 1)
     (in_bom yes) (on_board yes) (dnp no)
-    (property "Reference" "#PWR036" (at 176.53 92.71 0)
+    (property "Reference" "#PWR016" (at 176.53 92.71 0)
       (effects (font (size 1.27 1.27)) hide)
     )
@@
       (project "IVC-k30"
         (path "/dd13a6b9-cb24-4a73-96ce-c29930072fba/69e17b68-518f-4a96-bc5f-1d2df7d01a56"
-          (reference "#PWR036") (unit 1)
-        )
-      )
+          (reference "#PWR016") (unit 1)
+        )
+      )

Commit message: Committed changes to k30 board from Oct 9th 2023
Changed lines of the file:
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@@
     (stroke (width 0) (type default))
   )
-  (wire (pts (xy 88.9 165.1) (xy 106.68 165.1))
+  (wire (pts (xy 88.9 165.1) (xy 100.33 165.1))
     (stroke (width 0) (type default))
   )
@@
     (stroke (width 0) (type default))
   )
-  (wire (pts (xy 88.9 85.09) (xy 106.68 85.09))
+  (wire (pts (xy 88.9 85.09) (xy 100.33 85.09))
     (stroke (width 0) (type default))
   )
@@
     )
   )
-  (global_label "~{DS2}" (shape input) (at 106.68 85.09 0) (fields_autoplaced)
+  (global_label "~{DS2}" (shape input) (at 100.33 85.09 0) (fields_autoplaced)
     (effects (font (size 1.27 1.27)) (justify left))
-    (property "Intersheetrefs" "${INTERSHEET_REFS}" (at 0 0 0)
+    (property "Intersheetrefs" "${INTERSHEET_REFS}" (at -6.35 0 0)
       (effects (font (size 1.27 1.27)) hide)
     )
@@
     )
   )
-  (global_label "~{DS0}" (shape input) (at 106.68 165.1 0) (fields_autoplaced)
+  (global_label "~{DS0}" (shape input) (at 100.33 165.1 0) (fields_autoplaced)
     (effects (font (size 1.27 1.27)) (justify left))
-    (property "Intersheetrefs" "${INTERSHEET_REFS}" (at 0 0 0)
+    (property "Intersheetrefs" "${INTERSHEET_REFS}" (at -6.35 0 0)
       (effects (font (size 1.27 1.27)) hide)
     )
