File: hardware/IVC-STH7/Bus.kicad_sch (KiCad schematic)
At the start: 1 part, among them U10 Hirose PCN10-128P-2.54DS(72)

Commit message: STM32H7 PCB work in progress
Connections:
- net +12V: no longer names the net of U10.c31 (+12V)
- no-connect marks 2 -> 3
Changed lines of the file:
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@@
   (junction (at 43.18 19.05) (diameter 0) (color 0 0 0 0)
   )
+  (no_connect (at 234.95 100.33))
   (no_connect (at 71.12 100.33))
   (no_connect (at 147.32 100.33))
@@
     (stroke (width 0) (type default))
   )
-  (wire (pts (xy 205.74 100.33) (xy 234.95 100.33))
-    (stroke (width 0) (type default))
-  )
   (wire (pts (xy 135.89 31.75) (xy 147.32 31.75))
     (stroke (width 0) (type default))
@@
   )
   (wire (pts (xy 135.89 41.91) (xy 147.32 41.91))
-    (stroke (width 0) (type default))
-  )
-  (wire (pts (xy 205.74 99.06) (xy 205.74 100.33))
     (stroke (width 0) (type default))
   )
@@
         )
       )
-    )
-  )
-  (symbol (lib_id "power:+12V") (at 205.74 99.06 0) (unit 1)
-    (in_bom yes) (on_board yes) (dnp no)
-    (property "Reference" "#PWR0107" (at 205.74 102.87 0)
-      (effects (font (size 1.27 1.27)) hide)
-    )
-    (property "Value" "+12V" (at 205.74 95.25 0)
-      (effects (font (size 1.27 1.27)))
-    )
-    (property "Footprint" "" (at 205.74 99.06 0)
-      (effects (font (size 1.27 1.27)) hide)
-    )
-    (property "Datasheet" "" (at 205.74 99.06 0)
-      (effects (font (size 1.27 1.27)) hide)
-    )
-    (pin "1")
-    (instances
-      (project "IVC-STH7"
-        (path "/dd13a6b9-cb24-4a73-96ce-c29930072fba/372c1966-b642-4e1e-8b8f-ada6fd5e1159"
-          (reference "#PWR0107") (unit 1)
-        )
-      )
