File: hardware/IVC-STH7/IO.kicad_sch (KiCad schematic)
At the start: 43 parts, among them J2 Amphenol 10118194-0001LF, J5 SPI2, J6 USART1, J7 Hirose DM3D-S, J7 I^{2}C1, J8 USART2, J9 Bel SI-60062-F, U4 LAN8742A

Commit message: STM32H7 PCB work in progress
Connections:
- net TD-: now reaches J9.3 (TD-), R13.2, U4.20 (TXN)
- net TD+: now reaches J9.1 (TD+), R13.2, U4.21 (TXP)
- net RD-: now reaches J9.6 (RD-), R13.2, U4.22 (RXN)
- net RD+: now reaches J9.4 (RD+), R13.2, U4.23 (RXP)
Other:
- moved on the sheet: J5, J6, J7, J8, J9, JP4, JP5, JP6, JP7, R13, R14, R5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
