File: hardware/IVC-STH7/IVC-STH7.kicad_pcb (KiCad board)
At the start: 4 copper layers, 160 x 100 mm, 120 parts, among them J1 5V, J10 SPI2, J11 USART1, J12 I^{2}C1, J13 USART2, J2 5V, J3 3.3V, J4 5V, J5 3.3V, J6 Conn_ST_STDC14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

Commit message: STM32H7 PCB work in progress
Parts:
- moved JP1 78.5 mm to (77.2, 90.9), turned to 180 degrees
- moved R9 70.0 mm to (143.8, 53.3), turned to -135 degrees
- moved R22 26.7 mm to (105.2, 106.2), turned to 180 degrees
- moved C33 26.0 mm to (101.6, 98.0), turned to 90 degrees
- moved R20 25.5 mm to (105.2, 104.1), turned to 180 degrees
- moved R23 24.1 mm to (103.1, 112.3), turned to 90 degrees
- moved C31 22.2 mm to (84.3, 116.8), turned to 180 degrees
- moved R18 21.6 mm to (90.9, 112.3), turned to 90 degrees
- moved R19 20.0 mm to (101.1, 112.3), turned to 90 degrees
- moved R21 18.4 mm to (99.1, 112.3), turned to 90 degrees
- moved L2 17.8 mm to (84.3, 114.3), turned to 180 degrees
- moved R26 15.5 mm to (99.6, 98.0), turned to 90 degrees
- moved R28 14.8 mm to (93.5, 98.0), turned to -90 degrees
- moved R8 14.5 mm to (80.8, 89.4), turned to -90 degrees
- moved R24 14.1 mm to (91.4, 98.0), turned to 90 degrees
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Connections:
- net Net-(J9-RD+) renamed /IO/RD+
- net Net-(J9-RD-) renamed /IO/RD-
- net Net-(J9-TD+) renamed /IO/TD+
- net Net-(J9-TD-) renamed /IO/TD-
- U10 pad c31: +12V -> unconnected-(U10C-+12V-Padc31)
Routing:
- net GND: track 0.00 -> 122.6 mm, vias 0 -> 65
- net +3.3V: track 55.5 -> 177.9 mm, vias 0 -> 31
- net LD15: track 0.00 -> 96.1 mm, vias 0 -> 2
- net LA0: track 0.00 -> 87.3 mm, vias 0 -> 2
- net ~{VBR1}: track 0.00 -> 69.8 mm, vias 0 -> 2
- net LD13: track 0.00 -> 69.6 mm, vias 0 -> 2
- net LD12: track 0.00 -> 69.4 mm, vias 0 -> 2
- net LD14: track 0.00 -> 69.0 mm, vias 0 -> 2
- net LD11: track 0.00 -> 67.4 mm, vias 0 -> 2
- net ~{VBR2}: track 0.00 -> 66.5 mm, vias 0 -> 2
- net ~{VBR3}: track 0.00 -> 64.8 mm, vias 0 -> 2
- net RMII_TXEN: track 0.00 -> 57.4 mm
- net RMII_TXD1: track 0.00 -> 55.6 mm
- net LD4: track 0.00 -> 54.5 mm, vias 0 -> 2
- net LD5: track 0.00 -> 54.4 mm, vias 0 -> 2
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