File: controllers/bigboy/hardware/BigBoy/Controller.kicad_sch (KiCad schematic)
At the start: 10 parts, among them U2 STM32H743BITx, U6 KC3225Z25.0000C1KX00, Y1 32,768Hz

Commit message: Reorganized to make it easier to group hardware and firmware files together
Other:
- title: IVC-STH7 -> BigBoy
Changed lines of the file:
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@@
   (paper "A4")
   (title_block
-    (title "IVC-STH7")
+    (title "BigBoy")
     (rev "1")
   )
@@
         )
       )
-      (project "IVC-STH7"
+      (project "BigBoy"
         (path "/dd13a6b9-cb24-4a73-96ce-c29930072fba/69e17b68-518f-4a96-bc5f-1d2df7d01a56"
           (reference "R8") (unit 1)
@@
         )
       )
-      (project "IVC-STH7"
+      (project "BigBoy"
         (path "/dd13a6b9-cb24-4a73-96ce-c29930072fba/dfc443dd-7c5d-4956-9c53-a8ea419d150b"
           (reference "Y1") (unit 1)
@@
     (pin "94")
     (instances
-      (project "IVC-STH7"
+      (project "BigBoy"
         (path "/dd13a6b9-cb24-4a73-96ce-c29930072fba/dfc443dd-7c5d-4956-9c53-a8ea419d150b"
           (reference "U2") (unit 1)
@@
         )
       )
-      (project "IVC-STH7"
+      (project "BigBoy"
         (path "/dd13a6b9-cb24-4a73-96ce-c29930072fba/69e17b68-518f-4a96-bc5f-1d2df7d01a56"
           (reference "R8") (unit 1)
@@
         )
       )
-      (project "IVC-STH7"
+      (project "BigBoy"
         (path "/dd13a6b9-cb24-4a73-96ce-c29930072fba"
           (reference "U19") (unit 1)
@@
         )
       )
-      (project "IVC-STH7"
+      (project "BigBoy"
         (path "/dd13a6b9-cb24-4a73-96ce-c29930072fba/dfc443dd-7c5d-4956-9c53-a8ea419d150b"
           (reference "C27") (unit 1)
@@
         )
       )
-      (project "IVC-STH7"
+      (project "BigBoy"
         (path "/dd13a6b9-cb24-4a73-96ce-c29930072fba/dfc443dd-7c5d-4956-9c53-a8ea419d150b"
           (reference "C26") (unit 1)
@@
         )
       )
-      (project "IVC-STH7"
+      (project "BigBoy"
         (path "/dd13a6b9-cb24-4a73-96ce-c29930072fba/69e17b68-518f-4a96-bc5f-1d2df7d01a56"
           (reference "R8") (unit 1)
@@
         )
       )
-      (project "IVC-STH7"
+      (project "BigBoy"
         (path "/dd13a6b9-cb24-4a73-96ce-c29930072fba/dfc443dd-7c5d-4956-9c53-a8ea419d150b"
           (reference "#PWR035") (unit 1)
@@
         )
       )
-      (project "IVC-STH7"
+      (project "BigBoy"
         (path "/dd13a6b9-cb24-4a73-96ce-c29930072fba/69e17b68-518f-4a96-bc5f-1d2df7d01a56"
           (reference "R8") (unit 1)
@@
         )
       )
-      (project "IVC-STH7"
+      (project "BigBoy"
         (path "/dd13a6b9-cb24-4a73-96ce-c29930072fba"
           (reference "#PWR074") (unit 1)
@@
         )
       )
-      (project "IVC-STH7"
+      (project "BigBoy"
         (path "/dd13a6b9-cb24-4a73-96ce-c29930072fba"
           (reference "#PWR073") (unit 1)
@@
     (pin "94")
     (instances
-      (project "IVC-STH7"
+      (project "BigBoy"
         (path "/dd13a6b9-cb24-4a73-96ce-c29930072fba/dfc443dd-7c5d-4956-9c53-a8ea419d150b"
           (reference "U2") (unit 3)
@@
     (pin "94")
     (instances
-      (project "IVC-STH7"
+      (project "BigBoy"
         (path "/dd13a6b9-cb24-4a73-96ce-c29930072fba/dfc443dd-7c5d-4956-9c53-a8ea419d150b"
           (reference "U2") (unit 2)
@@
         )
       )
-      (project "IVC-STH7"
+      (project "BigBoy"
         (path "/dd13a6b9-cb24-4a73-96ce-c29930072fba"
           (reference "C15") (unit 1)

Commit message: Most of the routing for BigBoy is done
Parts:
- R13: value 51 -> 50
- U2: footprint Package_QFP:LQFP-208_28x28mm_P0.5mm -> Computie_SMT:LQFP-208_28x28mm_P0.5mm
Connections:
- net AH_DIR: now also U2.139 (PC7); no longer U2.54 (PA5)
- net UL2: now also U2.50 (PA3); no longer U2.138 (PC6)
- net UL3: now also U2.53 (PA4); no longer U2.139 (PC7)
- net ~{AH_OE}: now also U2.138 (PC6); no longer U2.50 (PA3)
- net ~{AL_OE}: now also U2.54 (PA5); no longer U2.53 (PA4)

Commit message: BigBoy Rev.1 is complete and ready to order
Parts:
- U2: footprint Computie_SMT:LQFP-208_28x28mm_P0.5mm -> Package_QFP:LQFP-208_28x28mm_P0.5mm
- Y1: footprint Crystal:Crystal_SMD_3225-4Pin_3.2x2.5mm_HandSoldering -> Crystal:Crystal_SMD_3215-2Pin_3.2x1.5mm
Connections:
- net CLK_25M: now also U2.32 (PH0); no longer U6.3 (CLK)
- net at R13.1: now also U6.3 (CLK); no longer U2.32 (PH0)
Other:
- moved on the sheet: C15, R13, U6
