File: vmebusboards/6-Slot-Backplane/Slot1.kicad_sch (KiCad schematic)
At the start: 20 parts, among them U1 74ACT32, U2 74ACT32, U5 VME-J1-4R-NS

Commit message: Updated
Parts:
- removed JP10: BG0, symbol Jumper:Jumper_2_Small_Bridged
- removed JP11: BG1, symbol Jumper:Jumper_2_Small_Bridged
- removed JP12: BG2, symbol Jumper:Jumper_2_Small_Bridged
- removed JP13: BG3, symbol Jumper:Jumper_2_Small_Bridged
- removed JP14: IACK, symbol Jumper:Jumper_2_Small_Bridged
- removed R10, R11, R12, R13, R9: 82k, symbol Device:R_Small
- removed U1, U2: 74ACT32, symbol 74xx:74LS32
- J1: renamed from U5; footprint Computie_Connectors:DIN41612_C_4x32_Male_Horizontal_THT -> Computie_Connectors:DIN41612_C_4x32_Female_Vertical_THT
- JP10: renamed from JP6; footprint (none) -> Connector_PinHeader_2.54mm:PinHeader_1x02_P2.54mm_Vertical
- JP11: renamed from JP7; footprint (none) -> Connector_PinHeader_2.54mm:PinHeader_1x02_P2.54mm_Vertical
- JP12: renamed from JP8; footprint (none) -> Connector_PinHeader_2.54mm:PinHeader_1x02_P2.54mm_Vertical
- JP13: renamed from JP9; footprint (none) -> Connector_PinHeader_2.54mm:PinHeader_1x02_P2.54mm_Vertical
- JP9: renamed from JP5; footprint (none) -> Connector_PinHeader_2.54mm:PinHeader_1x02_P2.54mm_Vertical
Other:
- moved on the sheet: JP10, JP11, JP12, JP13, JP9
