File: vmebusboards/6-Slot-Backplane/6-Slot-Backplane.kicad_sch (KiCad schematic)
At the start: 18 parts, among them J1 ATX-24, J2 +5V, J3 GND, J4 +12V, J5 -12V, J6 +5VStandby, J7 SYSTEM MONITOR, U1 74ACT32, U2 74ACT32

Commit message: Updated
Parts:
- added C25, C26, C27, C28, C29: 0.1uF, symbol Device:C_Small
- added U5, U6, U7, U8, U9: 74ACT32, Package_SO:SOIC-14_3.9x8.7mm_P1.27mm, symbol 74xx:74LS32
- C1: renamed from C3; footprint (none) -> Capacitor_THT:CP_Radial_D8.0mm_P5.00mm
- C3: renamed from C5; footprint (none) -> Capacitor_THT:CP_Radial_D8.0mm_P5.00mm
- C5: renamed from C7; footprint (none) -> Capacitor_THT:CP_Radial_D8.0mm_P5.00mm
- J107: renamed from J7; footprint (none) -> Connector_PinHeader_2.54mm:PinHeader_1x05_P2.54mm_Vertical; symbol Connector_Generic:Conn_01x04 -> Connector_Generic:Conn_01x05
- U3: renamed from U1; footprint (none) -> Package_SO:SOIC-14_3.9x8.7mm_P1.27mm
- U4: renamed from U2; footprint (none) -> Package_SO:SOIC-14_3.9x8.7mm_P1.27mm
- renumbered C4 to C2, C6 to C4, C8 to C6, C1 to C7, C2 to C8, J1 to J101, J2 to J102, J3 to J103, J4 to J104, J5 to J105, J6 to J106
Connections:
- net +5V: now also J107.4 (Pin_4), C25.1, C26.1, C27.1, C28.1, C29.1, U5.14 (VCC), U6.14 (VCC), U7.14 (VCC), U8.14 (VCC), U9.14 (VCC)
- net GND: now also J107.5 (Pin_5), C25.2, C26.2, C27.2, C28.2, C29.2, U5.7 (GND), U6.7 (GND), U7.7 (GND), U8.7 (GND), U9.7 (GND); no longer J107.4 (Pin_4)
Other:
- added sheet Slot3 (Slot3.kicad_sch)
- added sheet Slot4 (Slot4.kicad_sch)
- added sheet Slot5 (Slot5.kicad_sch)
- added sheet Slot6 (Slot6.kicad_sch)
- moved on the sheet: C1, C2, C3, C4, C5, C6, C7, C8, J101, J102, J103, J104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

Commit message: Added SystemBoardSMT, renamed k30 boards, and added progress
Parts:
- J101: footprint (none) -> Computie_Connectors:TE_1-1775099-3_ATX_24_Pin_PowerSupply
Changed lines of the file:
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@@
 			)
 		)
-		(property "Footprint" ""
+		(property "Footprint" "Computie_Connectors:TE_1-1775099-3_ATX_24_Pin_PowerSupply"
 			(at 33.02 39.37 0)
 			(effects
