File: vmebusboards/6-Slot-Backplane/Slot3.kicad_sch (KiCad schematic)
At the start: 15 parts, among them J2 VME-J1-4R-NS, U3 74ACT32, U4 74ACT32

Commit message: Updated
Parts:
- renumbered H3 to H5, H4 to H6, J2 to J3, JP14 to JP19, JP15 to JP20, JP16 to JP21, JP17 to JP22, JP18 to JP23, R15 to R10, R16 to R11, R17 to R12, R18 to R13, R14 to R9, U3 to U4, U4 to U5, U3 to U5
Connections:
- net ~{SLOT1_BG0IN}: now also U4.4; no longer U4.1
- net ~{SLOT1_BG0OUT}: now also U4.5; no longer U4.2
- net ~{SLOT1_BG1IN}: now also U4.9; no longer U4.4
- net ~{SLOT1_BG1OUT}: now also U4.10; no longer U4.5
- net ~{SLOT1_BG2IN}: now also U4.12; no longer U4.9
- net ~{SLOT1_BG2OUT}: now also U4.13; no longer U4.10
- net ~{SLOT1_BG3IN}: now also U5.1; no longer U5.12
- net ~{SLOT1_BG3OUT}: now also U5.2; no longer U5.13
- net ~{SLOT1_IACKIN}: now also U5.4; no longer U5.1
- net ~{SLOT1_IACKOUT}: now also U5.5; no longer U5.2
- net ~{SLOT2_BG0IN}: now also U4.6; no longer U4.3
- net ~{SLOT2_BG1IN}: now also U4.8; no longer U4.6
- net ~{SLOT2_BG2IN}: now also U4.11; no longer U4.8
- net ~{SLOT2_BG3IN}: now also U5.3; no longer U5.11
- net ~{SLOT2_IACKIN}: now also U5.6; no longer U5.3

Commit message: Added SystemBoardSMT, renamed k30 boards, and added progress
Parts:
- R10, R11, R12, R13, R9: footprint (none) -> Resistor_SMD:R_0805_2012Metric_Pad1.20x1.40mm_HandSolder
Changed lines of the file:
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@@
 			)
 		)
-		(property "Footprint" ""
+		(property "Footprint" "Resistor_SMD:R_0805_2012Metric_Pad1.20x1.40mm_HandSolder"
 			(at 127 190.5 0)
 			(effects
@@
 			)
 		)
-		(property "Footprint" ""
+		(property "Footprint" "Resistor_SMD:R_0805_2012Metric_Pad1.20x1.40mm_HandSolder"
 			(at 127 170.18 0)
 			(effects
@@
 			)
 		)
-		(property "Footprint" ""
+		(property "Footprint" "Resistor_SMD:R_0805_2012Metric_Pad1.20x1.40mm_HandSolder"
 			(at 127 149.86 0)
 			(effects
@@
 			)
 		)
-		(property "Footprint" ""
+		(property "Footprint" "Resistor_SMD:R_0805_2012Metric_Pad1.20x1.40mm_HandSolder"
 			(at 127 129.54 0)
 			(effects
@@
 			)
 		)
-		(property "Footprint" ""
+		(property "Footprint" "Resistor_SMD:R_0805_2012Metric_Pad1.20x1.40mm_HandSolder"
 			(at 196.85 129.54 0)
 			(effects
