File: vmebusboards/6-Slot-Backplane/Slot4.kicad_sch (KiCad schematic)
At the start: 15 parts, among them J2 VME-J1-4R-NS, U3 74ACT32, U4 74ACT32

Commit message: Updated
Parts:
- renumbered H3 to H7, H4 to H8, J2 to J4, JP14 to JP24, JP15 to JP25, JP16 to JP26, JP17 to JP27, JP18 to JP28, R14 to R23, R15 to R24, R16 to R25, R17 to R26, R18 to R27, U3 to U5, U4 to U6, U3 to U6
Connections:
- net ~{SLOT1_BG0IN}: now also U5.9; no longer U5.1
- net ~{SLOT1_BG0OUT}: now also U5.10; no longer U5.2
- net ~{SLOT1_BG1IN}: now also U5.12; no longer U5.4
- net ~{SLOT1_BG1OUT}: now also U5.13; no longer U5.5
- net ~{SLOT1_BG2IN}: now also U6.1; no longer U6.9
- net ~{SLOT1_BG2OUT}: now also U6.2; no longer U6.10
- net ~{SLOT1_BG3IN}: now also U6.4; no longer U6.12
- net ~{SLOT1_BG3OUT}: now also U6.5; no longer U6.13
- net ~{SLOT1_IACKIN}: now also U6.9; no longer U6.1
- net ~{SLOT1_IACKOUT}: now also U6.10; no longer U6.2
- net ~{SLOT2_BG0IN}: now also U5.8; no longer U5.3
- net ~{SLOT2_BG1IN}: now also U5.11; no longer U5.6
- net ~{SLOT2_BG2IN}: now also U6.3; no longer U6.8
- net ~{SLOT2_BG3IN}: now also U6.6; no longer U6.11
- net ~{SLOT2_IACKIN}: now also U6.8; no longer U6.3

Commit message: Added SystemBoardSMT, renamed k30 boards, and added progress
Parts:
- R23, R24, R25, R26, R27: footprint (none) -> Resistor_SMD:R_0805_2012Metric_Pad1.20x1.40mm_HandSolder
Changed lines of the file:
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@@
 			)
 		)
-		(property "Footprint" ""
+		(property "Footprint" "Resistor_SMD:R_0805_2012Metric_Pad1.20x1.40mm_HandSolder"
 			(at 127 190.5 0)
 			(effects
@@
 			)
 		)
-		(property "Footprint" ""
+		(property "Footprint" "Resistor_SMD:R_0805_2012Metric_Pad1.20x1.40mm_HandSolder"
 			(at 127 170.18 0)
 			(effects
@@
 			)
 		)
-		(property "Footprint" ""
+		(property "Footprint" "Resistor_SMD:R_0805_2012Metric_Pad1.20x1.40mm_HandSolder"
 			(at 127 149.86 0)
 			(effects
@@
 			)
 		)
-		(property "Footprint" ""
+		(property "Footprint" "Resistor_SMD:R_0805_2012Metric_Pad1.20x1.40mm_HandSolder"
 			(at 127 129.54 0)
 			(effects
@@
 			)
 		)
-		(property "Footprint" ""
+		(property "Footprint" "Resistor_SMD:R_0805_2012Metric_Pad1.20x1.40mm_HandSolder"
 			(at 196.85 129.54 0)
 			(effects
