File: vmebusboards/6-Slot-Backplane/Slot5.kicad_sch (KiCad schematic)
At the start: 15 parts, among them J2 VME-J1-4R-NS, U3 74ACT32, U4 74ACT32

Commit message: Updated
Parts:
- renumbered H4 to H10, H3 to H9, J2 to J5, JP14 to JP29, JP15 to JP30, JP16 to JP31, JP17 to JP32, JP18 to JP33, R14 to R28, R15 to R29, R16 to R30, R17 to R31, R18 to R32, U3 to U6, U4 to U7, U3 to U7
Connections:
- net ~{SLOT1_BG0IN}: now also U6.12; no longer U6.1
- net ~{SLOT1_BG0OUT}: now also U6.13; no longer U6.2
- net ~{SLOT1_BG1IN}: now also U7.1; no longer U7.4
- net ~{SLOT1_BG1OUT}: now also U7.2; no longer U7.5
- net ~{SLOT1_BG2IN}: now also U7.4; no longer U7.9
- net ~{SLOT1_BG2OUT}: now also U7.5; no longer U7.10
- net ~{SLOT1_BG3IN}: now also U7.9; no longer U7.12
- net ~{SLOT1_BG3OUT}: now also U7.10; no longer U7.13
- net ~{SLOT1_IACKIN}: now also U7.12; no longer U7.1
- net ~{SLOT1_IACKOUT}: now also U7.13; no longer U7.2
- net ~{SLOT2_BG0IN}: now also U6.11; no longer U6.3
- net ~{SLOT2_BG1IN}: now also U7.3; no longer U7.6
- net ~{SLOT2_BG2IN}: now also U7.6; no longer U7.8
- net ~{SLOT2_BG3IN}: now also U7.8; no longer U7.11
- net ~{SLOT2_IACKIN}: now also U7.11; no longer U7.3

Commit message: Added SystemBoardSMT, renamed k30 boards, and added progress
Parts:
- R28, R29, R30, R31, R32: footprint (none) -> Resistor_SMD:R_0805_2012Metric_Pad1.20x1.40mm_HandSolder
Changed lines of the file:
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@@
 			)
 		)
-		(property "Footprint" ""
+		(property "Footprint" "Resistor_SMD:R_0805_2012Metric_Pad1.20x1.40mm_HandSolder"
 			(at 127 190.5 0)
 			(effects
@@
 			)
 		)
-		(property "Footprint" ""
+		(property "Footprint" "Resistor_SMD:R_0805_2012Metric_Pad1.20x1.40mm_HandSolder"
 			(at 127 170.18 0)
 			(effects
@@
 			)
 		)
-		(property "Footprint" ""
+		(property "Footprint" "Resistor_SMD:R_0805_2012Metric_Pad1.20x1.40mm_HandSolder"
 			(at 127 149.86 0)
 			(effects
@@
 			)
 		)
-		(property "Footprint" ""
+		(property "Footprint" "Resistor_SMD:R_0805_2012Metric_Pad1.20x1.40mm_HandSolder"
 			(at 127 129.54 0)
 			(effects
@@
 			)
 		)
-		(property "Footprint" ""
+		(property "Footprint" "Resistor_SMD:R_0805_2012Metric_Pad1.20x1.40mm_HandSolder"
 			(at 196.85 129.54 0)
 			(effects
