File: vmebusboards/6-Slot-Backplane/Slot6.kicad_sch (KiCad schematic)
At the start: 15 parts, among them J2 VME-J1-4R-NS, U3 74ACT32, U4 74ACT32

Commit message: Updated
Parts:
- renumbered H3 to H11, H4 to H12, J2 to J6, JP14 to JP34, JP15 to JP35, JP16 to JP36, JP17 to JP37, JP18 to JP38, R14 to R33, R15 to R34, R16 to R35, R17 to R36, R18 to R37, U3 to U8, U4 to U9

Commit message: Added SystemBoardSMT, renamed k30 boards, and added progress
Parts:
- R33, R34, R35, R36, R37: footprint (none) -> Resistor_SMD:R_0805_2012Metric_Pad1.20x1.40mm_HandSolder
Changed lines of the file:
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@@
 			)
 		)
-		(property "Footprint" ""
+		(property "Footprint" "Resistor_SMD:R_0805_2012Metric_Pad1.20x1.40mm_HandSolder"
 			(at 127 190.5 0)
 			(effects
@@
 			)
 		)
-		(property "Footprint" ""
+		(property "Footprint" "Resistor_SMD:R_0805_2012Metric_Pad1.20x1.40mm_HandSolder"
 			(at 127 170.18 0)
 			(effects
@@
 			)
 		)
-		(property "Footprint" ""
+		(property "Footprint" "Resistor_SMD:R_0805_2012Metric_Pad1.20x1.40mm_HandSolder"
 			(at 127 149.86 0)
 			(effects
@@
 			)
 		)
-		(property "Footprint" ""
+		(property "Footprint" "Resistor_SMD:R_0805_2012Metric_Pad1.20x1.40mm_HandSolder"
 			(at 127 129.54 0)
 			(effects
@@
 			)
 		)
-		(property "Footprint" ""
+		(property "Footprint" "Resistor_SMD:R_0805_2012Metric_Pad1.20x1.40mm_HandSolder"
 			(at 196.85 129.54 0)
 			(effects
