File: vmebusboards/6-Slot-Backplane/6-Slot-Backplane.kicad_pcb (KiCad board)
At the start: 4 copper layers, 96 parts, among them J1 VME-J1-4R-NS, J107 SYSTEM MONITOR, J2 VME-J1-4R-NS, J3 VME-J1-4R-NS, J4 VME-J1-4R-NS, J5 VME-J1-4R-NS, J6 VME-J1-4R-NS, U3 74ACT32, U4 74ACT32, U5 74ACT32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

Commit message: Added SystemBoardSMT, renamed k30 boards, and added progress
Parts:
- added J101: ATX-24, Computie_Connectors:TE_1-1775099-3_ATX_24_Pin_PowerSupply, F.Cu at (230.5, 116.2)
- added R1: 470, Resistor_SMD:R_0805_2012Metric_Pad1.20x1.40mm_HandSolder, F.Cu at (202.8, 126.5)
- added R10: 82k, Resistor_SMD:R_0805_2012Metric_Pad1.20x1.40mm_HandSolder, F.Cu at (229.8, 129.5)
- added R11: 82k, Resistor_SMD:R_0805_2012Metric_Pad1.20x1.40mm_HandSolder, F.Cu at (229.8, 132.4)
- added R12: 82k, Resistor_SMD:R_0805_2012Metric_Pad1.20x1.40mm_HandSolder, F.Cu at (229.8, 135.4)
- added R13: 82k, Resistor_SMD:R_0805_2012Metric_Pad1.20x1.40mm_HandSolder, F.Cu at (229.8, 138.3)
- added R14: 82k, Resistor_SMD:R_0805_2012Metric_Pad1.20x1.40mm_HandSolder, F.Cu at (236.6, 126.5)
- added R15: 82k, Resistor_SMD:R_0805_2012Metric_Pad1.20x1.40mm_HandSolder, F.Cu at (236.6, 129.5)
- added R16: 82k, Resistor_SMD:R_0805_2012Metric_Pad1.20x1.40mm_HandSolder, F.Cu at (236.6, 132.4)
- added R17: 82k, Resistor_SMD:R_0805_2012Metric_Pad1.20x1.40mm_HandSolder, F.Cu at (236.6, 135.4)
- added R18: 82k, Resistor_SMD:R_0805_2012Metric_Pad1.20x1.40mm_HandSolder, F.Cu at (236.6, 138.3)
- added R19: 330, Resistor_SMD:R_0805_2012Metric_Pad1.20x1.40mm_HandSolder, F.Cu at (202.8, 138.3)
- added R2: 330, Resistor_SMD:R_0805_2012Metric_Pad1.20x1.40mm_HandSolder, F.Cu at (202.8, 129.5)
- added R20: 470, Resistor_SMD:R_0805_2012Metric_Pad1.20x1.40mm_HandSolder, F.Cu at (202.8, 141.3)
- added R21: 330, Resistor_SMD:R_0805_2012Metric_Pad1.20x1.40mm_HandSolder, F.Cu at (209.6, 138.3)
- added R22: 470, Resistor_SMD:R_0805_2012Metric_Pad1.20x1.40mm_HandSolder, F.Cu at (209.6, 141.3)
- added R23: 82k, Resistor_SMD:R_0805_2012Metric_Pad1.20x1.40mm_HandSolder, F.Cu at (223.1, 126.5)
- added R24: 82k, Resistor_SMD:R_0805_2012Metric_Pad1.20x1.40mm_HandSolder, F.Cu at (223.1, 129.5)
- added R25: 82k, Resistor_SMD:R_0805_2012Metric_Pad1.20x1.40mm_HandSolder, F.Cu at (223.1, 132.4)
- added R26: 82k, Resistor_SMD:R_0805_2012Metric_Pad1.20x1.40mm_HandSolder, F.Cu at (223.1, 135.4)
- added R27: 82k, Resistor_SMD:R_0805_2012Metric_Pad1.20x1.40mm_HandSolder, F.Cu at (223.1, 138.3)
- added R28: 82k, Resistor_SMD:R_0805_2012Metric_Pad1.20x1.40mm_HandSolder, F.Cu at (216.3, 126.5)
- added R29: 82k, Resistor_SMD:R_0805_2012Metric_Pad1.20x1.40mm_HandSolder, F.Cu at (216.3, 129.5)
- added R3: 330, Resistor_SMD:R_0805_2012Metric_Pad1.20x1.40mm_HandSolder, F.Cu at (202.8, 132.4)
- added R30: 82k, Resistor_SMD:R_0805_2012Metric_Pad1.20x1.40mm_HandSolder, F.Cu at (216.3, 132.4)
- added R31: 82k, Resistor_SMD:R_0805_2012Metric_Pad1.20x1.40mm_HandSolder, F.Cu at (216.3, 135.4)
- added R32: 82k, Resistor_SMD:R_0805_2012Metric_Pad1.20x1.40mm_HandSolder, F.Cu at (216.3, 138.3)
- added R33: 82k, Resistor_SMD:R_0805_2012Metric_Pad1.20x1.40mm_HandSolder, F.Cu at (243.3, 126.5)
- added R34: 82k, Resistor_SMD:R_0805_2012Metric_Pad1.20x1.40mm_HandSolder, F.Cu at (243.3, 129.5)
- added R35: 82k, Resistor_SMD:R_0805_2012Metric_Pad1.20x1.40mm_HandSolder, F.Cu at (243.3, 132.4)
- added R36: 82k, Resistor_SMD:R_0805_2012Metric_Pad1.20x1.40mm_HandSolder, F.Cu at (243.3, 135.4)
- added R37: 82k, Resistor_SMD:R_0805_2012Metric_Pad1.20x1.40mm_HandSolder, F.Cu at (243.3, 138.3)
- added R4: 470, Resistor_SMD:R_0805_2012Metric_Pad1.20x1.40mm_HandSolder, F.Cu at (202.8, 135.4)
- added R5: 330, Resistor_SMD:R_0805_2012Metric_Pad1.20x1.40mm_HandSolder, F.Cu at (209.6, 126.5)
- added R6: 470, Resistor_SMD:R_0805_2012Metric_Pad1.20x1.40mm_HandSolder, F.Cu at (209.6, 129.5)
- added R7: 330, Resistor_SMD:R_0805_2012Metric_Pad1.20x1.40mm_HandSolder, F.Cu at (209.6, 132.4)
- added R8: 470, Resistor_SMD:R_0805_2012Metric_Pad1.20x1.40mm_HandSolder, F.Cu at (209.6, 135.4)
- added R9: 82k, Resistor_SMD:R_0805_2012Metric_Pad1.20x1.40mm_HandSolder, F.Cu at (229.8, 126.5)
- added U1: TCA0372_Dual_OpAmp, Package_SO:SOIC-16W_7.5x10.3mm_P1.27mm, B.Cu at (28.7, 39.2)
- added U2: TCA0372_Dual_OpAmp, Package_SO:SOIC-16W_7.5x10.3mm_P1.27mm, B.Cu at (153.5, 39.2)
- RN1, RN10, RN11, RN12, RN13, RN14, RN15, RN16, RN17, RN18, RN19, RN2, RN20, RN21, RN22, RN23, RN24, RN3, RN4, RN5, RN6, RN7, RN8, RN9: footprint Resistor_THT:R_Array_SIP10 -> Connector_PinHeader_2.54mm:PinHeader_1x10_P2.54mm_Vertical
- moved JP18 196.5 mm to (-8.94, 111.9)
- moved JP17 190.0 mm to (-8.94, 106.8)
- moved JP16 183.6 mm to (-8.94, 101.8)
- moved JP15 177.2 mm to (-8.94, 96.7)
- moved JP14 170.8 mm to (-8.94, 91.6)
- moved U3 10.8 mm to (50.4, 70.5)
- moved U4 10.8 mm to (50.4, 83.0)
- moved U5 10.8 mm to (70.8, 70.5)
- moved U6 10.8 mm to (91.1, 70.5)
- moved U7 10.8 mm to (111.4, 70.5)
- moved U8 10.8 mm to (111.4, 83.0)
- moved U9 10.8 mm to (131.7, 70.5)
- turned RN1 to 0 degrees
- turned RN10 to 0 degrees
- turned RN11 to 0 degrees
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Routing:
- net D0: track 0.00 -> 63.5 mm
- net +5V: track 0.00 -> 42.4 mm
- net ~{BCLR}: track 0.00 -> 42.4 mm
- net ~{BBSY}: track 0.00 -> 42.4 mm
- net GND: track 0.00 -> 42.4 mm
- net D8: track 0.00 -> 42.4 mm
- net D1: track 0.00 -> 42.4 mm
- net D12: track 21.2 -> 0.00 mm
- net D9: track 0.00 -> 21.2 mm
- net A25: track 21.2 -> 0.00 mm
- net ~{SLOT1_BG0OUT}: track 0.00 -> 15.0 mm

Commit message: Reorganized a bit
Parts:
- moved J101 12.9 mm to (231.9, 103.4)
Changed lines of the file:
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@@
 	(footprint "Computie_Connectors:TE_1-1775099-3_ATX_24_Pin_PowerSupply"
 		(layer "F.Cu")
-		(at 230.502 116.1986)
+		(at 231.915 103.373)
 		(property "Reference" "J101"
 			(at -17.54785 -5.99281 0)
