File: vmebusboards/60mm-Extender/60mm-Extender.kicad_sch (KiCad schematic)
At the start: 2 parts, among them U1 VME64-P1-3R, U2 VME64-P1-3R

Commit message: Updated
Parts:
- U2: footprint Connector_DIN:DIN41612_R_3x32_Female_Horizontal_THT -> Computie_Connectors:DIN41612_R_3x32_Reverse_Female_Horizontal_THT
Changed lines of the file:
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@@
 			)
 		)
-		(property "Footprint" "Connector_DIN:DIN41612_R_3x32_Female_Horizontal_THT"
+		(property "Footprint" "Computie_Connectors:DIN41612_R_3x32_Reverse_Female_Horizontal_THT"
 			(at 162.56 109.22 0)
 			(effects
@@
 			)
 		)
-		(property "Footprint" "Connector_DIN:DIN41612_R_3x32_Female_Horizontal_THT"
+		(property "Footprint" "Computie_Connectors:DIN41612_R_3x32_Reverse_Female_Horizontal_THT"
 			(at 104.14 109.22 0)
 			(effects
@@
 			)
 		)
-		(property "Footprint" "Connector_DIN:DIN41612_R_3x32_Female_Horizontal_THT"
+		(property "Footprint" "Computie_Connectors:DIN41612_R_3x32_Reverse_Female_Horizontal_THT"
 			(at 49.53 109.22 0)
 			(effects

Commit message: Updating with more work in progress
Parts:
- J1: renamed from U2; value VME64-P1-3R -> VME64-J1-3R
- P1: renamed from U1; symbol Computie_Connectors:VME64-J1-3R -> Computie_Connectors:VME64-P1-3R
Changed lines of the file:
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@@
 		(on_board yes)
 		(dnp no)
-		(property "Reference" "#PWR02"
+		(property "Reference" "#PWR04"
 			(at 46.99 102.87 0)
 			(effects
@@
 			(project "60mm-Extender"
 				(path "/be3632b1-5a12-4f31-a97d-ef7119b241f9"
-					(reference "#PWR02")
+					(reference "#PWR04")
 					(unit 1)
 				)
@@
 		(dnp no)
 		(fields_autoplaced yes)
-		(property "Reference" "U2"
+		(property "Reference" "J1"
 			(at 173.99 149.8599 0)
 			(effects
@@
 			)
 		)
-		(property "Value" "VME64-P1-3R"
+		(property "Value" "VME64-J1-3R"
 			(at 173.99 152.3999 0)
 			(effects
@@
 			(project "60mm-Extender"
 				(path "/be3632b1-5a12-4f31-a97d-ef7119b241f9"
-					(reference "U2")
+					(reference "J1")
 					(unit 3)
 				)
@@
 	)
 	(symbol
-		(lib_id "Computie_Connectors:VME64-J1-3R")
+		(lib_id "Computie_Connectors:VME64-P1-3R")
 		(at 162.56 62.23 0)
 		(unit 3)
@@
 		(dnp no)
 		(fields_autoplaced yes)
-		(property "Reference" "U1"
+		(property "Reference" "P1"
 			(at 173.99 62.2299 0)
 			(effects
@@
 			)
 		)
-		(property "Description" "VME64 J1 (Backplane-side Socket), 3 Row DIN41612 Connector"
+		(property "Description" "VME64 P1 (Board-side Headers), 3 Row DIN41612 Connector"
 			(at 162.56 62.23 0)
 			(effects
@@
 			(project "60mm-Extender"
 				(path "/be3632b1-5a12-4f31-a97d-ef7119b241f9"
-					(reference "U1")
+					(reference "P1")
 					(unit 3)
 				)
@@
 		(dnp no)
 		(fields_autoplaced yes)
-		(property "Reference" "#PWR016"
+		(property "Reference" "#PWR03"
 			(at 46.99 100.33 0)
 			(effects
@@
 			(project "60mm-Extender"
 				(path "/be3632b1-5a12-4f31-a97d-ef7119b241f9"
-					(reference "#PWR016")
+					(reference "#PWR03")
 					(unit 1)
 				)
@@
 		(on_board yes)
 		(dnp no)
-		(property "Reference" "#PWR04"
+		(property "Reference" "#PWR08"
 			(at 91.44 80.01 0)
 			(effects
@@
 			(project "60mm-Extender"
 				(path "/be3632b1-5a12-4f31-a97d-ef7119b241f9"
-					(reference "#PWR04")
+					(reference "#PWR08")
 					(unit 1)
 				)
@@
 	)
 	(symbol
-		(lib_id "Computie_Connectors:VME64-J1-3R")
+		(lib_id "Computie_Connectors:VME64-P1-3R")
 		(at 104.14 62.23 0)
 		(unit 2)
@@
 		(dnp no)
 		(fields_autoplaced yes)
-		(property "Reference" "U1"
+		(property "Reference" "P1"
 			(at 115.57 62.2299 0)
 			(effects
@@
 			)
 		)
-		(property "Description" "VME64 J1 (Backplane-side Socket), 3 Row DIN41612 Connector"
+		(property "Description" "VME64 P1 (Board-side Headers), 3 Row DIN41612 Connector"
 			(at 104.14 62.23 0)
 			(effects
@@
 			(project "60mm-Extender"
 				(path "/be3632b1-5a12-4f31-a97d-ef7119b241f9"
-					(reference "U1")
+					(reference "P1")
 					(unit 2)
 				)
@@
 		(on_board yes)
 		(dnp no)
-		(property "Reference" "#PWR013"
+		(property "Reference" "#PWR016"
 			(at 149.86 132.08 0)
 			(effects
@@
 			(project "60mm-Extender"
 				(path "/be3632b1-5a12-4f31-a97d-ef7119b241f9"
-					(reference "#PWR013")
+					(reference "#PWR016")
 					(unit 1)
 				)
@@
 		(dnp no)
 		(fields_autoplaced yes)
-		(property "Reference" "#PWR015"
+		(property "Reference" "#PWR014"
 			(at 160.02 100.33 0)
 			(effects
@@
 			(project "60mm-Extender"
 				(path "/be3632b1-5a12-4f31-a97d-ef7119b241f9"
-					(reference "#PWR015")
+					(reference "#PWR014")
 					(unit 1)
 				)
@@
 		(dnp no)
 		(fields_autoplaced yes)
-		(property "Reference" "U2"
+		(property "Reference" "J1"
 			(at 115.57 149.8599 0)
 			(effects
@@
 			)
 		)
-		(property "Value" "VME64-P1-3R"
+		(property "Value" "VME64-J1-3R"
 			(at 115.57 152.3999 0)
 			(effects
@@
 			(project "60mm-Extender"
 				(path "/be3632b1-5a12-4f31-a97d-ef7119b241f9"
-					(reference "U2")
+					(reference "J1")
 					(unit 2)
 				)
@@
 	)
 	(symbol
-		(lib_id "Computie_Connectors:VME64-J1-3R")
+		(lib_id "Computie_Connectors:VME64-P1-3R")
 		(at 49.53 62.23 0)
 		(unit 1)
@@
 		(dnp no)
 		(fields_autoplaced yes)
-		(property "Reference" "U1"
+		(property "Reference" "P1"
 			(at 60.96 62.2299 0)
 			(effects
@@
 			)
 		)
-		(property "Description" "VME64 J1 (Backplane-side Socket), 3 Row DIN41612 Connector"
+		(property "Description" "VME64 P1 (Board-side Headers), 3 Row DIN41612 Connector"
 			(at 49.53 62.23 0)
 			(effects
@@
 			(project "60mm-Extender"
 				(path "/be3632b1-5a12-4f31-a97d-ef7119b241f9"
-					(reference "U1")
+					(reference "P1")
 					(unit 1)
 				)
@@
 		(on_board yes)
 		(dnp no)
-		(property "Reference" "#PWR07"
+		(property "Reference" "#PWR015"
 			(at 160.02 102.87 0)
 			(effects
@@
 			(project "60mm-Extender"
 				(path "/be3632b1-5a12-4f31-a97d-ef7119b241f9"
-					(reference "#PWR07")
+					(reference "#PWR015")
 					(unit 1)
 				)
@@
 		(on_board yes)
 		(dnp no)
-		(property "Reference" "#PWR06"
+		(property "Reference" "#PWR013"
 			(at 149.86 44.45 0)
 			(effects
@@
 			(project "60mm-Extender"
 				(path "/be3632b1-5a12-4f31-a97d-ef7119b241f9"
-					(reference "#PWR06")
+					(reference "#PWR013")
 					(unit 1)
 				)
@@
 		(on_board yes)
 		(dnp no)
-		(property "Reference" "#PWR09"
+		(property "Reference" "#PWR06"
 			(at 46.99 190.5 0)
 			(effects
@@
 			(project "60mm-Extender"
 				(path "/be3632b1-5a12-4f31-a97d-ef7119b241f9"
-					(reference "#PWR09")
+					(reference "#PWR06")
 					(unit 1)
 				)
@@
 		(on_board yes)
 		(dnp no)
-		(property "Reference" "#PWR05"
+		(property "Reference" "#PWR09"
 			(at 101.6 102.87 0)
 			(effects
@@
 			(project "60mm-Extender"
 				(path "/be3632b1-5a12-4f31-a97d-ef7119b241f9"
-					(reference "#PWR05")
+					(reference "#PWR09")
 					(unit 1)
 				)
@@
 		(on_board yes)
 		(dnp no)
-		(property "Reference" "#PWR08"
+		(property "Reference" "#PWR02"
 			(at 31.75 132.08 0)
 			(effects
@@
 			(project "60mm-Extender"
 				(path "/be3632b1-5a12-4f31-a97d-ef7119b241f9"
-					(reference "#PWR08")
+					(reference "#PWR02")
 					(unit 1)
 				)
@@
 		(on_board yes)
 		(dnp no)
-		(property "Reference" "#PWR014"
+		(property "Reference" "#PWR018"
 			(at 160.02 190.5 0)
 			(effects
@@
 			(project "60mm-Extender"
 				(path "/be3632b1-5a12-4f31-a97d-ef7119b241f9"
-					(reference "#PWR014")
+					(reference "#PWR018")
 					(unit 1)
 				)
@@
 		(on_board yes)
 		(dnp no)
-		(property "Reference" "#PWR03"
+		(property "Reference" "#PWR07"
 			(at 91.44 72.39 0)
 			(effects
@@
 			(project "60mm-Extender"
 				(path "/be3632b1-5a12-4f31-a97d-ef7119b241f9"
-					(reference "#PWR03")
+					(reference "#PWR07")
 					(unit 1)
 				)
@@
 		(dnp no)
 		(fields_autoplaced yes)
-		(property "Reference" "U2"
+		(property "Reference" "J1"
 			(at 60.96 149.8599 0)
 			(effects
@@
 			)
 		)
-		(property "Value" "VME64-P1-3R"
+		(property "Value" "VME64-J1-3R"
 			(at 60.96 152.3999 0)
 			(effects
@@
 			(project "60mm-Extender"
 				(path "/be3632b1-5a12-4f31-a97d-ef7119b241f9"
-					(reference "U2")
+					(reference "J1")
 					(unit 1)
 				)
@@
 		(dnp no)
 		(fields_autoplaced yes)
-		(property "Reference" "#PWR018"
+		(property "Reference" "#PWR05"
 			(at 46.99 187.96 0)
 			(effects
@@
 			(project "60mm-Extender"
 				(path "/be3632b1-5a12-4f31-a97d-ef7119b241f9"
-					(reference "#PWR018")
+					(reference "#PWR05")
 					(unit 1)
 				)
