File: vmebusboards/60mm-Extender/60mm-Extender.kicad_pcb (KiCad board)
At the start: 2 copper layers, 2 parts, among them U1 VME64-P1-3R, U2 VME64-P1-3R

Commit message: Updated
Parts:
- U2: footprint Connector_DIN:DIN41612_R_3x32_Female_Horizontal_THT -> Computie_Connectors:DIN41612_R_3x32_Reverse_Female_Horizontal_THT
- moved U2 28.7 mm to (49.5, 114.3)
- moved U1 11.7 mm to (97.5, 35.6)
Other:
- board outline added: 58.6 x 100 mm

Commit message: Updating with more work in progress
Parts:
- J1: renamed from U2; value VME64-P1-3R -> VME64-J1-3R
- moved P1 6.60 mm to (90.9, 35.6)
- renumbered U1 to P1
Routing:
- net GND: track 0.00 -> 320.9 mm
- net D0: track 0.00 -> 43.2 mm
- net ~{DS1}: track 0.00 -> 42.9 mm
- net D7: track 0.00 -> 42.9 mm
- net ~{IACKIN}: track 0.00 -> 42.9 mm
- net A5: track 0.00 -> 42.9 mm
- net A3: track 0.00 -> 42.9 mm
- net A2: track 0.00 -> 42.9 mm
- net A1: track 0.00 -> 42.9 mm
- net -12V: track 0.00 -> 42.9 mm
- net ~{IACKOUT}: track 0.00 -> 42.9 mm
- net ~{DS0}: track 0.00 -> 42.9 mm
- net SYSCLK: track 0.00 -> 42.9 mm
- net D5: track 0.00 -> 42.9 mm
- net D3: track 0.00 -> 42.9 mm
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Other:
- board size 58.6 x 100 mm -> 52 x 100 mm

Commit message: Reorganized a bit
Routing:
- net GND: track 320.9 -> 325.9 mm, vias 0 -> 9
- added copper zone on B.Cu, net GND
- added copper zone on F.Cu, net GND
Changed lines of the file:
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@@
 		(allow_soldermask_bridges_in_footprints no)
 		(pcbplotparams
-			(layerselection 0x00010fc_ffffffff)
+			(layerselection 0x00010f0_ffffffff)
 			(plot_on_all_layers_selection 0x0000000_00000000)
 			(disableapertmacros no)
@@
 			(outputformat 1)
 			(mirror no)
-			(drillshape 1)
+			(drillshape 0)
 			(scaleselection 1)
 			(outputdirectory "")
@@
 	(segment
 		(start 55.94164 90.551)
-		(end 84.328 90.551)
+		(end 70.104 90.551)
 		(width 0.2)
 		(layer "F.Cu")
@@
 	)
 	(segment
+		(start 50.8 92.71)
+		(end 47.752 92.71)
+		(width 0.2)
+		(layer "F.Cu")
+		(net 1)
+	)
+	(segment
 		(start 84.328 90.551)
 		(end 84.709 90.17)
@@
 	)
 	(segment
+		(start 52.07 91.44)
+		(end 50.8 92.71)
+		(width 0.2)
+		(layer "F.Cu")
+		(net 1)
+	)
+	(segment
 		(start 55.94164 82.931)
+		(end 70.104 82.931)
+		(width 0.2)
+		(layer "F.Cu")
+		(net 1)
+	)
+	(segment
+		(start 70.104 82.931)
 		(end 84.328 82.931)
 		(width 0.2)
@@
 	)
 	(segment
+		(start 70.104 90.551)
+		(end 84.328 90.551)
+		(width 0.2)
+		(layer "F.Cu")
+		(net 1)
+	)
+	(segment
 		(start 87.116 82.55)
 		(end 88.386 83.82)
@@
 		(net 1)
 	)
+	(via
+		(at 47.752 92.71)
+		(size 0.6)
+		(drill 0.3)
+		(layers "F.Cu" "B.Cu")
+		(net 1)
+	)
+	(via
+		(at 70.104 90.551)
+		(size 0.6)
+		(drill 0.3)
+		(layers "F.Cu" "B.Cu")
+		(net 1)
+	)
+	(via
+		(at 70.104 54.102)
+		(size 0.6)
+		(drill 0.3)
+		(layers "F.Cu" "B.Cu")
+		(net 1)
+	)
+	(via
+		(at 70.104 69.342)
+		(size 0.6)
+		(drill 0.3)
+		(layers "F.Cu" "B.Cu")
+		(net 1)
+	)
+	(via
+		(at 70.104 82.931)
+		(size 0.6)
+		(drill 0.3)
+		(layers "F.Cu" "B.Cu")
+		(net 1)
+	)
+	(via
+		(at 70.104 55.88)
+		(size 0.6)
+		(drill 0.3)
+		(layers "F.Cu" "B.Cu")
+		(net 1)
+	)
+	(via
+		(at 70.104 79.502)
+		(size 0.6)
+		(drill 0.3)
+		(layers "F.Cu" "B.Cu")
+		(net 1)
+	)
+	(via
+		(at 70.104 74.422)
+		(size 0.6)
+		(drill 0.3)
+		(layers "F.Cu" "B.Cu")
+		(net 1)
+	)
+	(via
+		(at 70.104 59.182)
+		(size 0.6)
+		(drill 0.3)
+		(layers "F.Cu" "B.Cu")
+		(net 1)
+	)
 	(segment
 		(start 55.753 54.61)
@@
 	(segment
 		(start 54.61 55.88)
-		(end 85.846 55.88)
+		(end 70.104 55.88)
 		(width 0.2)
 		(layer "B.Cu")
@@
 	)
 	(segment
+		(start 70.104 54.102)
+		(end 83.947 54.102)
+		(width 0.2)
+		(layer "B.Cu")
+		(net 1)
+	)
+	(segment
 		(start 49.53 55.88)
 		(end 50.8 54.61)
@@
 	(segment
 		(start 56.261 59.182)
-		(end 83.947 59.182)
+		(end 70.104 59.182)
+		(width 0.2)
+		(layer "B.Cu")
+		(net 1)
+	)
+	(segment
+		(start 70.104 74.422)
+		(end 83.947 74.422)
 		(width 0.2)
 		(layer "B.Cu")
@@
 	)
 	(segment
+		(start 70.104 79.502)
+		(end 83.947 79.502)
+		(width 0.2)
+		(layer "B.Cu")
+		(net 1)
+	)
+	(segment
 		(start 89.656 74.93)
 		(end 90.926 76.2)
@@
 	)
 	(segment
+		(start 70.104 59.182)
+		(end 83.947 59.182)
+		(width 0.2)
+		(layer "B.Cu")
+		(net 1)
+	)
+	(segment
 		(start 56.261 54.102)
-		(end 83.947 54.102)
+		(end 70.104 54.102)
+		(width 0.2)
+		(layer "B.Cu")
+		(net 1)
+	)
+	(segment
+		(start 69.977 69.342)
+		(end 70.104 69.215)
 		(width 0.2)
 		(layer "B.Cu")
@@
 	(segment
 		(start 56.261 74.422)
-		(end 83.947 74.422)
+		(end 70.104 74.422)
 		(width 0.2)
 		(layer "B.Cu")
@@
 	(segment
 		(start 56.261 69.342)
-		(end 83.947 69.342)
+		(end 69.977 69.342)
 		(width 0.2)
 		(layer "B.Cu")
@@
 	)
 	(segment
+		(start 70.231 69.342)
+		(end 83.947 69.342)
+		(width 0.2)
+		(layer "B.Cu")
+		(net 1)
+	)
+	(segment
 		(start 55.753 59.69)
 		(end 56.261 59.182)
@@
 	(segment
 		(start 56.261 79.502)
-		(end 83.947 79.502)
+		(end 70.104 79.502)
 		(width 0.2)
 		(layer "B.Cu")
@@
 	)
 	(segment
+		(start 70.104 55.88)
+		(end 85.846 55.88)
+		(width 0.2)
+		(layer "B.Cu")
+		(net 1)
+	)
+	(segment
 		(start 49.53 71.12)
 		(end 50.8 69.85)
@@
 	)
 	(segment
+		(start 70.104 69.215)
+		(end 70.231 69.342)
+		(width 0.2)
+		(layer "B.Cu")
+		(net 1)
+	)
+	(segment
 		(start 50.8 69.85)
 		(end 55.753 69.85)
@@
 		(net 87)
 	)
+	(zone
+		(net 1)
+		(net_name "GND")
+		(layer "F.Cu")
+		(hatch edge 0.5)
+		(connect_pads
+			(clearance 0.5)
+		)
+		(min_thickness 0.25)
+		(filled_areas_thickness no)
+		(fill yes
+			(thermal_gap 0.5)
+			(thermal_bridge_width 0.5)
+		)
+		(polygon
+			(pts
+				(xy 44.196 25.146) (xy 96.266 25.146) (xy 96.266 125.095) (xy 44.196 125.095)
+			)
+		)
+	)
+	(zone
+		(net 1)
+		(net_name "GND")
+		(layer "B.Cu")
+		(hatch edge 0.5)
+		(priority 1)
+		(connect_pads
+			(clearance 0.5)
+		)
+		(min_thickness 0.25)
+		(filled_areas_thickness no)
+		(fill yes
+			(thermal_gap 0.5)
+			(thermal_bridge_width 0.5)
+		)
+		(polygon
+			(pts
+				(xy 44.196 25.146) (xy 96.266 25.146) (xy 96.266 125.095) (xy 44.196 125.095)
+			)
+		)
+	)
 )
