File: vmebusboards/SystemBoardSMT/Bus.kicad_sch (KiCad schematic)
At the start: 1 part, among them U3 VME64-P1-3R

Commit message: Updating with more work in progress
Connections:
- no-connect marks 3 -> 13
Changed lines of the file:
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@@
 	)
 	(no_connect
+		(at 233.68 39.37)
+	)
+	(no_connect
+		(at 233.68 34.29)
+	)
+	(no_connect
+		(at 233.68 26.67)
+	)
+	(no_connect
+		(at 233.68 31.75)
+	)
+	(no_connect
 		(at 69.85 102.87)
 	)
 	(no_connect
+		(at 233.68 36.83)
+	)
+	(no_connect
+		(at 146.05 80.01)
+	)
+	(no_connect
+		(at 233.68 44.45)
+	)
+	(no_connect
+		(at 146.05 77.47)
+	)
+	(no_connect
+		(at 233.68 29.21)
+	)
+	(no_connect
+		(at 233.68 41.91)
+	)
+	(no_connect
 		(at 233.68 102.87)
 	)
@@
 			)
 		)
-		(property "Description" ""
+		(property "Description" "Power symbol creates a global label with name \"+5V\""
 			(at 144.78 105.41 0)
 			(effects
@@
 			)
 		)
-		(property "Description" ""
+		(property "Description" "Power symbol creates a global label with name \"+5V\""
 			(at 232.41 105.41 0)
 			(effects
@@
 			)
 		)
-		(property "Description" ""
+		(property "Description" "Power symbol creates a global label with name \"+5V\""
 			(at 68.58 105.41 0)
 			(effects
