File: vmebusboards/SystemBoardSMT/SystemBoardSMT.kicad_pcb (KiCad board)
At the start: 4 copper layers, 100 x 100 mm, 36 parts, among them J1 5V, J2 5V, J3 JTAG, SW1 RESET, U1 ATF1508AS-xxAx100, U2 74HC14, U3 VME64-P1-3R, Y1 Crystal

Commit message: Updating with more work in progress
Connections:
- U2 pad 1: (no net) -> unconnected-(U2-Pad1)
- U2 pad 10: (no net) -> unconnected-(U2-Pad10)
- U2 pad 11: (no net) -> unconnected-(U2-Pad11)
- U2 pad 12: (no net) -> unconnected-(U2-Pad12)
- U2 pad 13: (no net) -> unconnected-(U2-Pad13)
- U2 pad 2: (no net) -> unconnected-(U2-Pad2)
- U2 pad 8: (no net) -> unconnected-(U2-Pad8)
- U2 pad 9: (no net) -> unconnected-(U2-Pad9)
Changed lines of the file:
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@@
 	(net 108 "unconnected-(U1-I{slash}O-Pad52)")
 	(net 109 "unconnected-(U1-I{slash}OE2{slash}GCLK2-Pad90)")
+	(net 110 "unconnected-(U2-Pad8)")
+	(net 111 "unconnected-(U2-Pad9)")
+	(net 112 "unconnected-(U2-Pad1)")
+	(net 113 "unconnected-(U2-Pad10)")
+	(net 114 "unconnected-(U2-Pad13)")
+	(net 115 "unconnected-(U2-Pad12)")
+	(net 116 "unconnected-(U2-Pad2)")
+	(net 117 "unconnected-(U2-Pad11)")
 	(footprint "Connector_DIN:DIN41612_C_3x32_Male_Horizontal_THT"
 		(locked yes)
@@
 			(net 50 "unconnected-(U3B-SERCLK-Padb21)")
 			(pinfunction "SERCLK")
-			(pintype "bidirectional")
+			(pintype "bidirectional+no_connect")
 		)
 		(pad "b22" thru_hole circle
@@
 			(net 43 "unconnected-(U3B-SERDAT-Padb22)")
 			(pinfunction "SERDAT")
-			(pintype "bidirectional")
+			(pintype "bidirectional+no_connect")
 		)
 		(pad "b23" thru_hole circle
@@
 			(net 47 "unconnected-(U3C-D08-Padc1)")
 			(pinfunction "D08")
-			(pintype "bidirectional")
+			(pintype "bidirectional+no_connect")
 		)
 		(pad "c2" thru_hole circle
@@
 			(net 48 "unconnected-(U3C-D09-Padc2)")
 			(pinfunction "D09")
-			(pintype "bidirectional")
+			(pintype "bidirectional+no_connect")
 		)
 		(pad "c3" thru_hole circle
@@
 			(net 49 "unconnected-(U3C-D10-Padc3)")
 			(pinfunction "D10")
-			(pintype "bidirectional")
+			(pintype "bidirectional+no_connect")
 		)
 		(pad "c4" thru_hole circle
@@
 			(net 54 "unconnected-(U3C-D11-Padc4)")
 			(pinfunction "D11")
-			(pintype "bidirectional")
+			(pintype "bidirectional+no_connect")
 		)
 		(pad "c5" thru_hole circle
@@
 			(net 53 "unconnected-(U3C-D12-Padc5)")
 			(pinfunction "D12")
-			(pintype "bidirectional")
+			(pintype "bidirectional+no_connect")
 		)
 		(pad "c6" thru_hole circle
@@
 			(net 56 "unconnected-(U3C-D13-Padc6)")
 			(pinfunction "D13")
-			(pintype "bidirectional")
+			(pintype "bidirectional+no_connect")
 		)
 		(pad "c7" thru_hole circle
@@
 			(net 46 "unconnected-(U3C-D14-Padc7)")
 			(pinfunction "D14")
-			(pintype "bidirectional")
+			(pintype "bidirectional+no_connect")
 		)
 		(pad "c8" thru_hole circle
@@
 			(net 42 "unconnected-(U3C-D15-Padc8)")
 			(pinfunction "D15")
-			(pintype "bidirectional")
+			(pintype "bidirectional+no_connect")
 		)
 		(pad "c9" thru_hole circle
@@
 		(tags "capacitor handsolder")
 		(property "Reference" "C7"
-			(at 0 -1.68 360)
+			(at 0 -1.68 0)
 			(layer "F.SilkS")
 			(effects
@@
 		)
 		(property "Value" "0.1uF"
-			(at 0 1.68 360)
+			(at 0 1.68 0)
 			(layer "F.Fab")
 			(effects
@@
 		)
 		(fp_text user "${REFERENCE}"
-			(at 0 0 360)
+			(at 0 0 0)
 			(layer "F.Fab")
 			(effects
@@
 			(net 106 "unconnected-(U1-I{slash}O-Pad21)")
 			(pinfunction "I/O")
-			(pintype "bidirectional")
+			(pintype "bidirectional+no_connect")
 		)
 		(pad "22" smd roundrect
@@
 			(net 107 "unconnected-(U1-I{slash}O-Pad22)")
 			(pinfunction "I/O")
-			(pintype "bidirectional")
+			(pintype "bidirectional+no_connect")
 		)
 		(pad "23" smd roundrect
@@
 			(net 108 "unconnected-(U1-I{slash}O-Pad52)")
 			(pinfunction "I/O")
-			(pintype "bidirectional")
+			(pintype "bidirectional+no_connect")
 		)
 		(pad "53" smd roundrect
@@
 			(net 100 "unconnected-(U1-I{slash}OE1-Pad88)")
 			(pinfunction "I/OE1")
-			(pintype "input")
+			(pintype "input+no_connect")
 		)
 		(pad "89" smd roundrect
@@
 			(net 109 "unconnected-(U1-I{slash}OE2{slash}GCLK2-Pad90)")
 			(pinfunction "I/OE2/GCLK2")
-			(pintype "input")
+			(pintype "input+no_connect")
 		)
 		(pad "91" smd roundrect
@@
 			(layers "F.Cu" "F.Paste" "F.Mask")
 			(roundrect_rratio 0.25)
+			(net 112 "unconnected-(U2-Pad1)")
+			(pintype "input+no_connect")
 		)
 		(pad "2" smd roundrect
@@
 			(layers "F.Cu" "F.Paste" "F.Mask")
 			(roundrect_rratio 0.25)
+			(net 116 "unconnected-(U2-Pad2)")
+			(pintype "output+no_connect")
 		)
 		(pad "3" smd roundrect
@@
 			(layers "F.Cu" "F.Paste" "F.Mask")
 			(roundrect_rratio 0.25)
+			(net 110 "unconnected-(U2-Pad8)")
+			(pintype "output+no_connect")
 		)
 		(pad "9" smd roundrect
@@
 			(layers "F.Cu" "F.Paste" "F.Mask")
 			(roundrect_rratio 0.25)
+			(net 111 "unconnected-(U2-Pad9)")
+			(pintype "input+no_connect")
 		)
 		(pad "10" smd roundrect
@@
 			(layers "F.Cu" "F.Paste" "F.Mask")
 			(roundrect_rratio 0.25)
+			(net 113 "unconnected-(U2-Pad10)")
+			(pintype "output+no_connect")
 		)
 		(pad "11" smd roundrect
@@
 			(layers "F.Cu" "F.Paste" "F.Mask")
 			(roundrect_rratio 0.25)
+			(net 117 "unconnected-(U2-Pad11)")
+			(pintype "input+no_connect")
 		)
 		(pad "12" smd roundrect
@@
 			(layers "F.Cu" "F.Paste" "F.Mask")
 			(roundrect_rratio 0.25)
+			(net 115 "unconnected-(U2-Pad12)")
+			(pintype "output+no_connect")
 		)
 		(pad "13" smd roundrect
@@
 			(layers "F.Cu" "F.Paste" "F.Mask")
 			(roundrect_rratio 0.25)
+			(net 114 "unconnected-(U2-Pad13)")
+			(pintype "input+no_connect")
 		)
 		(pad "14" smd roundrect
