File: vmebusboards/SystemBoardSMT/SystemBoardSMT.kicad_sch (KiCad schematic)
At the start: 35 parts, among them J1 5V, J2 5V, J3 JTAG, SW1 RESET, U1 ATF1508AS-xxAx100, U2 74HC14, Y1 Crystal

Commit message: Updating with more work in progress
Parts:
- added unit 6 of U2
- added unit 4 of U2
- added unit 5 of U2
- added unit 1 of U2
Connections:
- no-connect marks 3 -> 16
Other:
- note added: "UNUSED GATES"
