File: controllers/computie-vme/hardware/k30p-VME/k30p-VME.kicad_pcb (KiCad board)
At the start: 4 copper layers, 160 x 100 mm, 112 parts, among them J1 5V, J2 5V, J3 JTAG, J4 Serial1, J5 Serial2, P1 VME64-P1-3R, SW1 ~{RESET}, SW2 E-Switch TL2243, U1 MC68030RC, U10 FT231XS, U11 74ABT16245DL, U12 74ABT16245DL, U13 74ABT16245DL, U14 74ABT16245DL, U15 74ABT16245DL, U16 74HC148, U17 74LS30, U2 74HC14, U3 74HC05, U4 ATF1508AS-xxAx100, U5 AS6C8016, U6 AS6C8016, U7 AM29F040, U8 MC68681, U9 FT231XS, Y1 Crystal, Y2 Crystal

Commit message: WIP on k30p-VME
Parts:
- removed TP2: IPEND, TestPoint:TestPoint_THTPad_2.0x2.0mm_Drill1.0mm
- removed TP3: REFILL, TestPoint:TestPoint_THTPad_2.0x2.0mm_Drill1.0mm
- removed TP4: STATUS, TestPoint:TestPoint_THTPad_2.0x2.0mm_Drill1.0mm
- moved U17 61.2 mm to (146.6, 85.9)
- moved C15 54.4 mm to (137.6, 37.3)
- moved U6 54.4 mm to (146.6, 48.0)
- moved U7 53.6 mm to (147.8, 99.8)
- moved C13 53.4 mm to (146.6, 91.4)
- moved C17 50.4 mm to (96.3, 95.2), turned to 180 degrees
- moved C22 32.9 mm to (125.2, 95.2)
- moved RN2 23.1 mm to (82.5, 37.3)
- moved C19 22.4 mm to (96.3, 110.5), turned to 180 degrees
- moved C16 19.5 mm to (89.4, 64.5), turned to -90 degrees
- moved RN1 13.1 mm to (82.5, 40.6), turned to 0 degrees
- moved JP5 11.7 mm to (119.5, 117.6)
- moved JP6 11.7 mm to (123.2, 117.6)
- moved JP7 11.7 mm to (126.9, 117.6)
- moved JP8 11.7 mm to (130.6, 117.6)
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Connections:
- U1 pad E13: Net-(U1-IPEND) -> unconnected-(U1-IPEND-PadE13)
- U1 pad J12: Net-(U1-STATUS) -> unconnected-(U1-STATUS-PadJ12)
- U1 pad J13: Net-(U1-REFILL) -> unconnected-(U1-REFILL-PadJ13)
- U12 pad 11: LA22 -> LA30
- U12 pad 12: LA23 -> LA31
- U12 pad 13: LA24 -> LA16
- U12 pad 14: LA25 -> LA17
- U12 pad 16: LA26 -> LA18
- U12 pad 17: LA27 -> LA19
- U12 pad 19: LA28 -> LA20
- U12 pad 2: LA16 -> LA24
- U12 pad 20: LA29 -> LA21
- U12 pad 22: LA30 -> LA22
- U12 pad 23: LA31 -> LA23
- U12 pad 25: ~{A40X_OE} -> ~{AL_OE}
- U12 pad 26: VD15 -> VA23
- U12 pad 27: VD14 -> VA22
- U12 pad 29: VD13 -> VA21
- U12 pad 3: LA17 -> LA25
- U12 pad 30: VD12 -> VA20
- U12 pad 32: VD11 -> VA19
- U12 pad 33: VD10 -> VA18
- U12 pad 35: VD9 -> VA17
- U12 pad 36: VD8 -> VA16
- U12 pad 37: VA23 -> VD15
- U12 pad 38: VA22 -> VD14
- U12 pad 40: VA21 -> VD13
- U12 pad 41: VA20 -> VD12
- U12 pad 43: VA19 -> VD11
- U12 pad 44: VA18 -> VD10
- U12 pad 46: VA17 -> VD9
- U12 pad 47: VA16 -> VD8
- U12 pad 48: ~{AL_OE} -> ~{A40X_OE}
- U12 pad 5: LA18 -> LA26
- U12 pad 6: LA19 -> LA27
- U12 pad 8: LA20 -> LA28
- U12 pad 9: LA21 -> LA29
Routing:
- net LA4: track 0.00 -> 98.9 mm
- net LA3: track 0.00 -> 97.2 mm
- net LA2: track 0.00 -> 91.4 mm
- net LA1: track 0.00 -> 86.9 mm
- net +5V: track 0.00 -> 82.2 mm, vias 0 -> 4
- net ~{WR}: track 0.00 -> 81.0 mm, vias 0 -> 2
- net LD3: track 0.00 -> 76.7 mm, vias 0 -> 1
- net LD1: track 0.00 -> 72.1 mm
- net LD2: track 0.00 -> 71.1 mm
- net LD0: track 0.00 -> 67.6 mm
- net FC0: track 0.00 -> 67.4 mm
- net ~{BGACK}: track 0.00 -> 64.7 mm
- net ~{DSACK0}: track 0.00 -> 64.3 mm, vias 0 -> 1
- net FC2: track 0.00 -> 59.6 mm
- net ~{RESET}: track 0.00 -> 57.9 mm, vias 0 -> 1
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
Commit message: k30p-VME PCB work in progress
Parts:
- added RN3: CAT16-103J4LF, Resistor_SMD:R_Cat16-4, F.Cu at (92.3, 37.3)
- added RN4: CAT16-103J4LF, Resistor_SMD:R_Cat16-4, F.Cu at (96.5, 37.3)
- C13: moved to B.Cu
- RN1, RN2: value 10k -> CAT16-103J4LF; footprint Resistor_THT:R_Array_SIP9 -> Resistor_SMD:R_Cat16-4
- moved JP1 86.7 mm to (137.4, 122.7)
- moved JP2 86.7 mm to (141.1, 122.7)
- moved U17 55.0 mm to (119.2, 38.3)
- moved U11 15.9 mm to (171.4, 90.8)
- moved U15 15.9 mm to (171.4, 106.7)
- moved C13 13.5 mm to (146.6, 104.9)
- moved U7 7.41 mm to (141.5, 103.6), turned to 90 degrees
- moved RN2 5.49 mm to (88.0, 37.3), turned to 90 degrees
- moved C17 3.68 mm to (96.3, 91.6)
- moved C22 3.68 mm to (125.2, 91.6)
- moved C19 3.68 mm to (96.3, 106.8)
- moved C21 3.68 mm to (125.2, 106.8)
- moved RN1 3.53 mm to (83.8, 37.3), turned to 90 degrees
- moved U4 3.05 mm to (110.7, 100.1)
- moved C30 2.41 mm to (114.6, 59.7)
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Connections:
- RN1 pad 1: +5V -> ~{BGACK}
- RN1 pad 2: ~{BGACK} -> ~{AVEC}
- RN1 pad 3: ~{AVEC} -> ~{BERR}
- RN1 pad 4: ~{BERR} -> ~{DSACK0}
- RN1 pad 5: ~{DSACK0} -> +5V
- RN1 pad 6: ~{DSACK1} -> +5V
- RN1 pad 7: Net-(RN1-R6) -> +5V
- RN1 pad 8: Net-(RN1-R7) -> +5V
- RN2 pad 1: +5V -> ~{DSACK1}
- RN2 pad 2: ~{BR} -> Net-(RN2-R2.1)
- RN2 pad 3: ~{RESET} -> Net-(RN2-R3.1)
- RN2 pad 4: ~{IPL0} -> Net-(RN2-R4.1)
- RN2 pad 5: ~{IPL1} -> +5V
- RN2 pad 6: ~{IPL2} -> +5V
- RN2 pad 7: ~{MMUDIS} -> +5V
- RN2 pad 8: ~{CDIS} -> +5V
- U1 pad G1: Net-(RN1-R6) -> Net-(RN2-R2.1)
- U1 pad J1: Net-(RN1-R7) -> Net-(RN2-R3.1)
- U1 pad L1: Net-(RN1-R8) -> Net-(RN2-R4.1)
- U11 pad 2: LA0 -> unconnected-(U11-B0-Pad2)
- U11 pad 47: VA0 -> unconnected-(U11-A0-Pad47)
- U15 pad 47: VA0 -> ~{VLWORD}
Routing:
- net LA19: track 21.9 -> 158.1 mm, vias 0 -> 6
- net LA20: track 26.7 -> 160.2 mm, vias 0 -> 6
- net LD16: track 15.3 -> 133.2 mm, vias 0 -> 5
- net LA31: track 45.0 -> 149.3 mm, vias 1 -> 2
- net LD31: track 70.2 -> 174.4 mm, vias 0 -> 4
- net LA18: track 27.2 -> 131.2 mm, vias 0 -> 5
- net LA30: track 42.1 -> 144.5 mm, vias 1 -> 2
- net LA17: track 18.4 -> 117.4 mm, vias 0 -> 5
- net LD30: track 73.1 -> 170.8 mm, vias 0 -> 4
- net LA16: track 21.7 -> 118.0 mm, vias 0 -> 4
- net LA29: track 38.7 -> 133.7 mm, vias 0 -> 1
- net LA15: track 15.3 -> 110.1 mm, vias 0 -> 3
- net LA28: track 34.9 -> 127.4 mm, vias 0 -> 1
- net LA27: track 36.9 -> 125.9 mm, vias 0 -> 1
- net LA26: track 32.6 -> 119.9 mm, vias 0 -> 1
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