File: controllers/computie-vme/hardware/k30p-VME/CPU.kicad_sch (KiCad schematic)
At the start: 17 parts, among them SW1 ~{RESET}, U1 MC68030RC, U2 74HC14, U3 74HC05

Commit message: k30p-VME rev.1, MemBird Woodcock rev.1, and frontpanels
Changed lines of the file:
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@@
 	(bus
 		(pts
-			(xy 43.18 16.51) (xy 27.94 16.51)
+			(xy 43.18 17.78) (xy 34.29 17.78)
 		)
 		(stroke
@@
 	(bus
 		(pts
-			(xy 36.83 22.86) (xy 36.83 104.14)
+			(xy 36.83 24.13) (xy 36.83 104.14)
 		)
 		(stroke
@@
 	(bus
 		(pts
-			(xy 43.18 16.51) (xy 43.18 21.59)
+			(xy 43.18 17.78) (xy 43.18 21.59)
 		)
 		(stroke
@@
 	(bus
 		(pts
-			(xy 36.83 22.86) (xy 27.94 22.86)
+			(xy 36.83 24.13) (xy 34.29 24.13)
 		)
 		(stroke
@@
 				)
 				(justify left)
-				(hide yes)
 			)
 		)
@@
 				)
 				(justify left)
-				(hide yes)
 			)
 		)
@@
 				)
 				(justify left)
-				(hide yes)
 			)
 		)
@@
 					(size 1.27 1.27)
 				)
-				(hide yes)
 			)
 		)
@@
 				)
 				(justify left)
-				(hide yes)
 			)
 		)
@@
 				)
 				(justify left)
-				(hide yes)
 			)
 		)
@@
 				)
 				(justify left)
-				(hide yes)
 			)
 		)
@@
 				)
 				(justify left)
-				(hide yes)
 			)
 		)
@@
 				)
 				(justify left)
-				(hide yes)
 			)
 		)
@@
 				)
 				(justify left)
-				(hide yes)
 			)
 		)
@@
 				)
 				(justify right)
-				(hide yes)
 			)
 		)
@@
 				)
 				(justify left)
-				(hide yes)
 			)
 		)
@@
 				)
 				(justify left)
-				(hide yes)
 			)
 		)
@@
 				)
 				(justify left)
-				(hide yes)
 			)
 		)
@@
 				)
 				(justify left)
-				(hide yes)
 			)
 		)
@@
 				)
 				(justify left)
-				(hide yes)
 			)
 		)
@@
 				)
 				(justify left)
-				(hide yes)
 			)
 		)
@@
 				)
 				(justify left)
-				(hide yes)
 			)
 		)
@@
 				)
 				(justify left)
-				(hide yes)
 			)
 		)
@@
 				)
 				(justify left)
-				(hide yes)
 			)
 		)
@@
 				)
 				(justify left)
-				(hide yes)
 			)
 		)
@@
 				)
 				(justify left)
-				(hide yes)
 			)
 		)
@@
 				)
 				(justify left)
-				(hide yes)
 			)
 		)
@@
 				)
 				(justify left)
-				(hide yes)
 			)
 		)
@@
 	(global_label "LA[0..31]"
 		(shape output)
-		(at 27.94 16.51 180)
+		(at 34.29 17.78 180)
 		(fields_autoplaced yes)
 		(effects
@@
 		)
 		(property "Intersheetrefs" "${INTERSHEET_REFS}"
-			(at 16.3066 16.51 0)
+			(at 22.6566 17.78 0)
 			(effects
 				(font
@@
 				)
 				(justify right)
-				(hide yes)
 			)
 		)
@@
 				)
 				(justify left)
-				(hide yes)
 			)
 		)
@@
 					(size 1.27 1.27)
 				)
-				(hide yes)
 			)
 		)
@@
 				)
 				(justify left)
-				(hide yes)
 			)
 		)
@@
 				)
 				(justify right)
-				(hide yes)
 			)
 		)
@@
 				)
 				(justify left)
-				(hide yes)
 			)
 		)
@@
 				)
 				(justify left)
-				(hide yes)
 			)
 		)
@@
 	(global_label "LD[0..31]"
 		(shape bidirectional)
-		(at 27.94 22.86 180)
+		(at 34.29 24.13 180)
 		(fields_autoplaced yes)
 		(effects
@@
 		)
 		(property "Intersheetrefs" "${INTERSHEET_REFS}"
-			(at 15.0139 22.86 0)
+			(at 21.3639 24.13 0)
 			(effects
 				(font
@@
 				)
 				(justify right)
-				(hide yes)
 			)
 		)
@@
 				)
 				(justify left)
-				(hide yes)
 			)
 		)
@@
 				)
 				(justify left)
-				(hide yes)
 			)
 		)
