File: controllers/computie-vme/hardware/k30p-VME/Memory.kicad_sch (KiCad schematic)
At the start: 3 parts, among them U5 AS6C8016, U6 AS6C8016, U7 AM29F040

Commit message: Updating with more work in progress
Other:
- note added: "BOOT FLASH"
- note added: "LOCAL STATIC RAM"
- title: k30-VME32 -> k30p-VME
- moved on the sheet: U5, U6, U7

Commit message: Basic systemboard logic for bus arbitration is working and tested
Parts:
- U5, U6: symbol Computie_Memory:AS6C8016 -> Computie_Memory:AS6C8016-55ZIN
- U7: symbol Computie_Memory:AM29F040 -> Computie_Memory:AM29F040-J
Connections:
- net A0 renamed LA0
- net A1 renamed LA1
- net A10 renamed LA10
- net A11 renamed LA11
- net A12 renamed LA12
- net A13 renamed LA13
- net A14 renamed LA14
- net A15 renamed LA15
- net A16 renamed LA16
- net A17 renamed LA17
- net A18 renamed LA18
- net A19 renamed LA19
- net A2 renamed LA2
- net A20 renamed LA20
- net A3 renamed LA3
- net A4 renamed LA4
- net A5 renamed LA5
- net A6 renamed LA6
- net A7 renamed LA7
- net A8 renamed LA8
- net A9 renamed LA9
- net D0 renamed LD0
- net D1 renamed LD1
- net D10 renamed LD10
- net D11 renamed LD11
- net D12 renamed LD12
- net D13 renamed LD13
- net D14 renamed LD14
- net D15 renamed LD15
- net D16 renamed LD16
- net D17 renamed LD17
- net D18 renamed LD18
- net D19 renamed LD19
- net D2 renamed LD2
- net D20 renamed LD20
- net D21 renamed LD21
- net D22 renamed LD22
- net D23 renamed LD23
- net D24 renamed LD24
- net D25 renamed LD25
- net D26 renamed LD26
- net D27 renamed LD27
- net D28 renamed LD28
- net D29 renamed LD29
- net D3 renamed LD3
- net D30 renamed LD30
- net D31 renamed LD31
- net D4 renamed LD4
- net D5 renamed LD5
- net D6 renamed LD6
- net D7 renamed LD7
- net D8 renamed LD8
- net D9 renamed LD9

Commit message: k30p-VME rev.1, MemBird Woodcock rev.1, and frontpanels
Changed lines of the file:
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@@
 	(bus
 		(pts
-			(xy 54.61 30.48) (xy 31.75 30.48)
+			(xy 54.61 30.48) (xy 39.37 30.48)
 		)
 		(stroke
@@
 	(bus
 		(pts
-			(xy 97.79 26.67) (xy 31.75 26.67)
+			(xy 97.79 26.67) (xy 39.37 26.67)
 		)
 		(stroke
@@
 		)
 	)
-	(global_label "~{WR}"
+	(global_label "~{RAMSEL}"
 		(shape input)
-		(at 100.33 88.9 0)
+		(at 100.33 83.82 0)
 		(fields_autoplaced yes)
 		(effects
@@
 		)
 		(property "Intersheetrefs" "${INTERSHEET_REFS}"
-			(at 0 6.35 0)
+			(at 110.5118 83.82 0)
 			(effects
 				(font
 					(size 1.27 1.27)
 				)
-				(hide yes)
-			)
-		)
-	)
-	(global_label "~{WR}"
+				(justify left)
+			)
+		)
+	)
+	(global_label "~{RAMSEL}"
 		(shape input)
-		(at 100.33 168.91 0)
+		(at 100.33 163.83 0)
 		(fields_autoplaced yes)
 		(effects
@@
 		)
 		(property "Intersheetrefs" "${INTERSHEET_REFS}"
-			(at 0 6.35 0)
+			(at 110.5118 163.83 0)
 			(effects
 				(font
 					(size 1.27 1.27)
 				)
-				(hide yes)
-			)
-		)
-	)
-	(global_label "~{RD}"
+				(justify left)
+			)
+		)
+	)
+	(global_label "~{DS3}"
 		(shape input)
-		(at 200.66 67.31 0)
+		(at 100.33 93.98 0)
 		(fields_autoplaced yes)
 		(effects
@@
 		)
 		(property "Intersheetrefs" "${INTERSHEET_REFS}"
-			(at 0 6.35 0)
+			(at 107.0042 93.98 0)
 			(effects
 				(font
 					(size 1.27 1.27)
 				)
-				(hide yes)
-			)
-		)
-	)
-	(global_label "~{DS2}"
+				(justify left)
+			)
+		)
+	)
+	(global_label "~{RD}"
 		(shape input)
-		(at 100.33 91.44 0)
+		(at 100.33 166.37 0)
 		(fields_autoplaced yes)
 		(effects
@@
 		)
 		(property "Intersheetrefs" "${INTERSHEET_REFS}"
-			(at -6.35 6.35 0)
+			(at 105.8552 166.37 0)
 			(effects
 				(font
 					(size 1.27 1.27)
 				)
-				(hide yes)
-			)
-		)
-	)
-	(global_label "~{ROMSEL}"
+				(justify left)
+			)
+		)
+	)
+	(global_label "~{DS2}"
 		(shape input)
-		(at 200.66 64.77 0)
+		(at 100.33 91.44 0)
 		(fields_autoplaced yes)
 		(effects
@@
 		)
 		(property "Intersheetrefs" "${INTERSHEET_REFS}"
-			(at 0 6.35 0)
+			(at 107.0042 91.44 0)
 			(effects
 				(font
 					(size 1.27 1.27)
 				)
-				(hide yes)
-			)
-		)
-	)
-	(global_label "~{DS0}"
+				(justify left)
+			)
+		)
+	)
+	(global_label "~{DS1}"
 		(shape input)
-		(at 100.33 171.45 0)
+		(at 100.33 173.99 0)
 		(fields_autoplaced yes)
 		(effects
@@
 		)
 		(property "Intersheetrefs" "${INTERSHEET_REFS}"
-			(at -6.35 6.35 0)
+			(at 107.0042 173.99 0)
 			(effects
 				(font
 					(size 1.27 1.27)
 				)
-				(hide yes)
-			)
-		)
-	)
-	(global_label "~{RAMSEL}"
+				(justify left)
+			)
+		)
+	)
+	(global_label "~{DS0}"
 		(shape input)
-		(at 100.33 163.83 0)
+		(at 100.33 171.45 0)
 		(fields_autoplaced yes)
 		(effects
@@
 		)
 		(property "Intersheetrefs" "${INTERSHEET_REFS}"
-			(at 0 6.35 0)
+			(at 107.0042 171.45 0)
 			(effects
 				(font
 					(size 1.27 1.27)
 				)
-				(hide yes)
-			)
-		)
-	)
-	(global_label "~{RD}"
+				(justify left)
+			)
+		)
+	)
+	(global_label "~{WR}"
 		(shape input)
-		(at 100.33 166.37 0)
+		(at 100.33 168.91 0)
 		(fields_autoplaced yes)
 		(effects
@@
 		)
 		(property "Intersheetrefs" "${INTERSHEET_REFS}"
-			(at 0 6.35 0)
+			(at 106.0366 168.91 0)
 			(effects
 				(font
 					(size 1.27 1.27)
 				)
-				(hide yes)
-			)
-		)
-	)
-	(global_label "~{DS3}"
+				(justify left)
+			)
+		)
+	)
+	(global_label "~{WR}"
 		(shape input)
-		(at 100.33 93.98 0)
+		(at 100.33 88.9 0)
 		(fields_autoplaced yes)
 		(effects
@@
 		)
 		(property "Intersheetrefs" "${INTERSHEET_REFS}"
-			(at 0 6.35 0)
+			(at 106.0366 88.9 0)
 			(effects
 				(font
 					(size 1.27 1.27)
 				)
-				(hide yes)
-			)
-		)
-	)
-	(global_label "~{RAMSEL}"
+				(justify left)
+			)
+		)
+	)
+	(global_label "~{WR}"
 		(shape input)
-		(at 100.33 83.82 0)
+		(at 200.66 69.85 0)
 		(fields_autoplaced yes)
 		(effects
@@
 		)
 		(property "Intersheetrefs" "${INTERSHEET_REFS}"
-			(at 0 6.35 0)
+			(at 206.3666 69.85 0)
 			(effects
 				(font
 					(size 1.27 1.27)
 				)
-				(hide yes)
-			)
-		)
-	)
-	(global_label "~{DS1}"
+				(justify left)
+			)
+		)
+	)
+	(global_label "~{RD}"
 		(shape input)
-		(at 100.33 173.99 0)
+		(at 200.66 67.31 0)
 		(fields_autoplaced yes)
 		(effects
@@
 		)
 		(property "Intersheetrefs" "${INTERSHEET_REFS}"
-			(at 0 6.35 0)
+			(at 206.1852 67.31 0)
 			(effects
 				(font
 					(size 1.27 1.27)
 				)
-				(hide yes)
+				(justify left)
 			)
 		)
@@
 	(global_label "LA[0..31]"
 		(shape input)
-		(at 31.75 30.48 180)
+		(at 39.37 30.48 180)
 		(fields_autoplaced yes)
 		(effects
@@
 		)
 		(property "Intersheetrefs" "${INTERSHEET_REFS}"
-			(at 20.1166 30.48 0)
+			(at 27.7366 30.48 0)
 			(effects
 				(font
@@
 				)
 				(justify right)
-				(hide yes)
+			)
+		)
+	)
+	(global_label "~{RD}"
+		(shape input)
+		(at 100.33 86.36 0)
+		(fields_autoplaced yes)
+		(effects
+			(font
+				(size 1.27 1.27)
+			)
+			(justify left)
+		)
+		(property "Intersheetrefs" "${INTERSHEET_REFS}"
+			(at 105.8552 86.36 0)
+			(effects
+				(font
+					(size 1.27 1.27)
+				)
+				(justify left)
 			)
 		)
@@
 	(global_label "LD[0..31]"
 		(shape bidirectional)
-		(at 31.75 26.67 180)
+		(at 39.37 26.67 180)
 		(fields_autoplaced yes)
 		(effects
@@
 		)
 		(property "Intersheetrefs" "${INTERSHEET_REFS}"
-			(at 18.8239 26.67 0)
+			(at 26.4439 26.67 0)
 			(effects
 				(font
@@
 				)
 				(justify right)
-				(hide yes)
-			)
-		)
-	)
-	(global_label "~{RD}"
+			)
+		)
+	)
+	(global_label "~{ROMSEL}"
 		(shape input)
-		(at 100.33 86.36 0)
+		(at 200.66 64.77 0)
 		(fields_autoplaced yes)
 		(effects
@@
 		)
 		(property "Intersheetrefs" "${INTERSHEET_REFS}"
-			(at 0 6.35 0)
+			(at 211.0837 64.77 0)
 			(effects
 				(font
 					(size 1.27 1.27)
 				)
-				(hide yes)
-			)
-		)
-	)
-	(global_label "~{WR}"
-		(shape input)
-		(at 200.66 69.85 0)
-		(fields_autoplaced yes)
-		(effects
-			(font
-				(size 1.27 1.27)
-			)
-			(justify left)
-		)
-		(property "Intersheetrefs" "${INTERSHEET_REFS}"
-			(at 0 6.35 0)
-			(effects
-				(font
-					(size 1.27 1.27)
-				)
-				(hide yes)
-			)
-		)
+				(justify left)
+			)
+		)
