File: controllers/computie-vme/hardware/k30p-VME/Transceivers.kicad_sch (KiCad schematic)
At the start: 5 parts, among them U10 74ABT16245DL, U11 74ABT16245DL, U12 74ABT16245DL, U14 74ABT16245DL, U16 74ABT16245DL

Commit message: Updating with more work in progress
Connections:
- net AL_DIR is gone; now on net GND: U10.1 (DIR1), U10.24 (DIR2)
Other:
- title: k30-VME32 -> k30p-VME
Changed lines of the file:
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@@
 	(paper "A4")
 	(title_block
-		(title "k30-VME32")
+		(title "k30p-VME")
 		(rev "1")
 	)
@@
 	)
 	(junction
+		(at 39.37 43.18)
+		(diameter 0)
+		(color 0 0 0 0)
+	)
+	(junction
 		(at 39.37 121.92)
 		(diameter 0)
@@
 	)
 	(junction
-		(at 40.64 43.18)
-		(diameter 0)
-		(color 0 0 0 0)
-	)
-	(junction
 		(at 101.6 43.18)
 		(diameter 0)
@@
 	(wire
 		(pts
+			(xy 39.37 43.18) (xy 41.91 43.18)
+		)
+		(stroke
+			(width 0)
+			(type default)
+		)
+	)
+	(wire
+		(pts
 			(xy 67.31 66.04) (xy 78.74 66.04)
 		)
@@
 	(wire
 		(pts
-			(xy 38.1 43.18) (xy 40.64 43.18)
+			(xy 39.37 40.64) (xy 35.56 40.64)
 		)
 		(stroke
@@
 	(wire
 		(pts
-			(xy 41.91 45.72) (xy 40.64 45.72)
-		)
-		(stroke
-			(width 0)
-			(type default)
-		)
-	)
-	(wire
-		(pts
 			(xy 67.31 88.9) (xy 78.74 88.9)
 		)
@@
 		)
 	)
+	(wire
+		(pts
+			(xy 39.37 45.72) (xy 39.37 43.18)
+		)
+		(stroke
+			(width 0)
+			(type default)
+		)
+	)
 	(bus
 		(pts
@@
 	(wire
 		(pts
+			(xy 39.37 43.18) (xy 39.37 40.64)
+		)
+		(stroke
+			(width 0)
+			(type default)
+		)
+	)
+	(wire
+		(pts
 			(xy 67.31 139.7) (xy 78.74 139.7)
 		)
@@
 	(wire
 		(pts
-			(xy 40.64 43.18) (xy 41.91 43.18)
-		)
-		(stroke
-			(width 0)
-			(type default)
-		)
-	)
-	(wire
-		(pts
 			(xy 41.91 144.78) (xy 30.48 144.78)
 		)
@@
 		)
 	)
+	(wire
+		(pts
+			(xy 35.56 40.64) (xy 35.56 41.91)
+		)
+		(stroke
+			(width 0)
+			(type default)
+		)
+	)
 	(bus
 		(pts
@@
 	(wire
 		(pts
+			(xy 41.91 45.72) (xy 39.37 45.72)
+		)
+		(stroke
+			(width 0)
+			(type default)
+		)
+	)
+	(wire
+		(pts
 			(xy 163.83 63.5) (xy 152.4 63.5)
 		)
@@
 	(wire
 		(pts
-			(xy 40.64 45.72) (xy 40.64 43.18)
-		)
-		(stroke
-			(width 0)
-			(type default)
-		)
-	)
-	(wire
-		(pts
 			(xy 67.31 83.82) (xy 78.74 83.82)
 		)
@@
 		)
 	)
-	(text_box "DURING THE FOLLOWING TRANSACTIONS:\nA16, A24:		ADDRESS LOW & ADDRESS HIGH ARE ACTIVE\nA40:			ADDRESS LOW, ADDRESS HIGH, & A40 CROSS ARE ACTIVE\nD8E, D8O, D16:	D16 CROSS IS ACTIVE, DSACK1 = L, DSACK0 = H\nMD32:			DATA LOW & MD32 CROSS ARE ACTIVE, DSACK1 = L, DSACK0 = L\n\n"
+	(text_box "DURING THE FOLLOWING TRANSACTIONS:\nA16, A24:		ADDRESS LOW & ADDRESS HIGH ARE ACTIVE\nA40:			ADDRESS LOW, ADDRESS HIGH, & A40 CROSS ARE ACTIVE\nD8E, D8O, D16:	D16 CROSS IS ACTIVE, DSACK1 = L, DSACK0 = H\nMD32:			DATA LOW & MD32 CROSS ARE ACTIVE, DSACK1 = L, DSACK0 = L\n				(NOTE: D32 IS NOT SUPPORTED ON 3U 3R VME)\n\n"
 		(exclude_from_sim no)
 		(at 127 128.27 0)
-		(size 87.63 12.7)
+		(size 87.63 13.97)
 		(stroke
 			(width 0)
@@
 		)
 	)
-	(global_label "AL_DIR"
-		(shape input)
-		(at 38.1 43.18 180)
-		(fields_autoplaced yes)
-		(effects
-			(font
-				(size 1.27 1.27)
-			)
-			(justify right)
-		)
-		(property "Intersheetrefs" "${INTERSHEET_REFS}"
-			(at 28.8857 43.18 0)
-			(effects
-				(font
-					(size 1.27 1.27)
-				)
-				(justify right)
-				(hide yes)
-			)
-		)
-	)
 	(global_label "~{DL_OE}"
 		(shape input)
@@
 					(unit 1)
 				)
+			)
+		)
+	)
+	(symbol
+		(lib_id "power:GND")
+		(at 35.56 41.91 0)
+		(unit 1)
+		(exclude_from_sim no)
+		(in_bom yes)
+		(on_board yes)
+		(dnp no)
+		(property "Reference" "#PWR046"
+			(at 35.56 48.26 0)
+			(effects
+				(font
+					(size 1.27 1.27)
+				)
+				(hide yes)
+			)
+		)
+		(property "Value" "GND"
+			(at 35.687 46.3042 0)
+			(effects
+				(font
+					(size 1.27 1.27)
+				)
+			)
+		)
+		(property "Footprint" ""
+			(at 35.56 41.91 0)
+			(effects
+				(font
+					(size 1.27 1.27)
+				)
+				(hide yes)
+			)
+		)
+		(property "Datasheet" ""
+			(at 35.56 41.91 0)
+			(effects
+				(font
+					(size 1.27 1.27)
+				)
+				(hide yes)
+			)
+		)
+		(property "Description" ""
+			(at 35.56 41.91 0)
+			(effects
+				(font
+					(size 1.27 1.27)
+				)
+				(hide yes)
+			)
+		)
+		(pin "1"
+		)
+		(instances
+			(project "k30p-VME"
+				(path "/dd13a6b9-cb24-4a73-96ce-c29930072fba/d84460b0-5709-47d7-8f66-71b9360a0384"
+					(reference "#PWR046")
+					(unit 1)
+				)

Commit message: Reorganized a bit
Other:
- note added: "A24 / A40 CROSS TRANSCEIVER"
- note removed: "ADDRESS HIGH / A40 CROSS TRANSCEIVER"
- moved on the sheet: U12, U14, U16

Commit message: Basic systemboard logic for bus arbitration is working and tested
Other:
- note added: "NOTE: ON THIS BOARD, D[7..0] ARE ALLOWED TO FLOAT HIGH DURING AN A40 CYCLE, INSTEAD OF BEING DRIVEN HIGH, TO SAVE A TRANSCEIVER"
- note removed: "NOTE: D[7..0] ARE ALLOWED TO FLOAT HIGH DURING AN A40 CYCLE, INSTEAD OF BEING DRIVEN HIGH, TO SAVE A TRANSCEIVER"
Changed lines of the file:
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@@
 	)
 	(image
-		(at 30.988 180.848)
-		(scale 0.162652)
+		(at 230.886 117.602)
+		(scale 0.427374)
 		(data "iVBORw0KGgoAAAANSUhEUgAABHsAAAEwCAIAAAColOqxAAAAA3NCSVQICAjb4U/gAAAACXBIWXMA"
 			"ABg4AAAYOAFT1w/+AAAgAElEQVR4nOydZ1wUyfPwa1lYYEGSBBUUMKCoKIIJ9FBREQQTBg5FwZ8B"
@@
 		)
 	)
-	(text "NOTE: D[7..0] ARE ALLOWED TO FLOAT HIGH DURING AN A40\nCYCLE, INSTEAD OF BEING DRIVEN HIGH, TO SAVE A TRANSCEIVER"
+	(text "NOTE: ON THIS BOARD, D[7..0] ARE ALLOWED TO FLOAT HIGH DURING AN A40\nCYCLE, INSTEAD OF BEING DRIVEN HIGH, TO SAVE A TRANSCEIVER"
 		(exclude_from_sim no)
-		(at 16.002 188.976 0)
+		(at 191.008 131.064 0)
 		(effects
 			(font
@@
 	(text "See VME64 Table 2-28"
 		(exclude_from_sim no)
-		(at 27.432 174.498 0)
+		(at 202.692 105.664 0)
 		(effects
 			(font
@@
 			)
 		)
-		(property "Datasheet" "https://assets.nexperia.com/documents/data-sheet/74ALVC164245.pdf"
+		(property "Datasheet" "https://www.ti.com/lit/ds/symlink/sn74abt16245a.pdf"
 			(at 54.61 146.05 0)
 			(effects
@@
 			)
 		)
-		(property "Description" ""
+		(property "Description" "Power symbol creates a global label with name \"GND\" , ground"
 			(at 121.92 93.98 0)
 			(effects
@@
 			)
 		)
-		(property "Description" ""
+		(property "Description" "Power symbol creates a global label with name \"+5V\""
 			(at 191.77 33.02 0)
 			(effects
@@
 			)
 		)
-		(property "Datasheet" "https://assets.nexperia.com/documents/data-sheet/74ALVC164245.pdf"
+		(property "Datasheet" "https://www.ti.com/lit/ds/symlink/sn74abt16245a.pdf"
 			(at 121.92 67.31 0)
 			(effects
@@
 			)
 		)
-		(property "Description" ""
+		(property "Description" "Power symbol creates a global label with name \"GND\" , ground"
 			(at 121.92 172.72 0)
 			(effects
@@
 			)
 		)
-		(property "Datasheet" "https://assets.nexperia.com/documents/data-sheet/74ALVC164245.pdf"
+		(property "Datasheet" "https://www.ti.com/lit/ds/symlink/sn74abt16245a.pdf"
 			(at 54.61 67.31 0)
 			(effects
@@
 			)
 		)
-		(property "Description" ""
+		(property "Description" "Power symbol creates a global label with name \"+5V\""
 			(at 121.92 111.76 0)
 			(effects
@@
 			)
 		)
-		(property "Description" ""
+		(property "Description" "Power symbol creates a global label with name \"+5V\""
 			(at 121.92 33.02 0)
 			(effects
@@
 			)
 		)
-		(property "Description" ""
+		(property "Description" "Power symbol creates a global label with name \"GND\" , ground"
 			(at 54.61 93.98 0)
 			(effects
@@
 			)
 		)
-		(property "Datasheet" "https://assets.nexperia.com/documents/data-sheet/74ALVC164245.pdf"
+		(property "Datasheet" "https://www.ti.com/lit/ds/symlink/sn74abt16245a.pdf"
 			(at 121.92 146.05 0)
 			(effects
@@
 			)
 		)
-		(property "Description" ""
+		(property "Description" "Power symbol creates a global label with name \"GND\" , ground"
 			(at 35.56 120.65 0)
 			(effects
@@
 			)
 		)
-		(property "Description" ""
+		(property "Description" "Power symbol creates a global label with name \"GND\" , ground"
 			(at 191.77 93.98 0)
 			(effects
@@
 			)
 		)
-		(property "Description" ""
+		(property "Description" "Power symbol creates a global label with name \"+5V\""
 			(at 54.61 33.02 0)
 			(effects
@@
 			)
 		)
-		(property "Description" ""
+		(property "Description" "Power symbol creates a global label with name \"GND\" , ground"
 			(at 54.61 172.72 0)
 			(effects
@@
 			)
 		)
-		(property "Description" ""
+		(property "Description" "Power symbol creates a global label with name \"GND\" , ground"
 			(at 35.56 41.91 0)
 			(effects
@@
 			)
 		)
-		(property "Description" ""
+		(property "Description" "Power symbol creates a global label with name \"+5V\""
 			(at 54.61 111.76 0)
 			(effects
@@
 			)
 		)
-		(property "Datasheet" "https://assets.nexperia.com/documents/data-sheet/74ALVC164245.pdf"
+		(property "Datasheet" "https://www.ti.com/lit/ds/symlink/sn74abt16245a.pdf"
 			(at 191.77 67.31 0)
 			(effects

Commit message: WIP on k30p-VME
Connections:
- net LA16: now also U11.13 (B8); no longer U11.2 (B0)
- net LA17: now also U11.14 (B9); no longer U11.3 (B1)
- net LA18: now also U11.16 (B10); no longer U11.5 (B2)
- net LA19: now also U11.17 (B11); no longer U11.6 (B3)
- net LA20: now also U11.19 (B12); no longer U11.8 (B4)
- net LA21: now also U11.20 (B13); no longer U11.9 (B5)
- net LA22: now also U11.22 (B14); no longer U11.11 (B6)
- net LA23: now also U11.23 (B15); no longer U11.12 (B7)
- net LA24: now also U11.2 (B0); no longer U11.13 (B8)
- net LA25: now also U11.3 (B1); no longer U11.14 (B9)
- net LA26: now also U11.5 (B2); no longer U11.16 (B10)
- net LA27: now also U11.6 (B3); no longer U11.17 (B11)
- net LA28: now also U11.8 (B4); no longer U11.19 (B12)
- net LA29: now also U11.9 (B5); no longer U11.20 (B13)
- net LA30: now also U11.11 (B6); no longer U11.22 (B14)
- net LA31: now also U11.12 (B7); no longer U11.23 (B15)
- net VA16: now also U11.36 (A8); no longer U11.47 (A0)
- net VA17: now also U11.35 (A9); no longer U11.46 (A1)
- net VA18: now also U11.33 (A10); no longer U11.44 (A2)
- net VA19: now also U11.32 (A11); no longer U11.43 (A3)
- net VA20: now also U11.30 (A12); no longer U11.41 (A4)
- net VA21: now also U11.29 (A13); no longer U11.40 (A5)
- net VA22: now also U11.27 (A14); no longer U11.38 (A6)
- net VA23: now also U11.26 (A15); no longer U11.37 (A7)
- net VD10: now also U11.44 (A2); no longer U11.33 (A10)
- net VD11: now also U11.43 (A3); no longer U11.32 (A11)
- net VD12: now also U11.41 (A4); no longer U11.30 (A12)
- net VD13: now also U11.40 (A5); no longer U11.29 (A13)
- net VD14: now also U11.38 (A6); no longer U11.27 (A14)
- net VD15: now also U11.37 (A7); no longer U11.26 (A15)
- net VD8: now also U11.47 (A0); no longer U11.36 (A8)
- net VD9: now also U11.46 (A1); no longer U11.35 (A9)
- net ~{A40X_OE}: now also U11.48 (~{OE1}); no longer U11.25 (~{OE2})
- net ~{AL_OE}: now also U11.25 (~{OE2}); no longer U11.48 (~{OE1})
Other:
- note added: "NOTE: THE UPPER AND LOWER UNITS ARE OPPOSITE TO SIMPLIFY THE PCB LAYOUT"

Commit message: k30p-VME PCB work in progress
Connections:
- net LA0: no longer names the net of U10.2 (B0)
- net VA0: no longer names the net of U10.47 (A0)
- net VA0: no longer U16.47 (A0)
- new net ~{VLWORD}: U16.47 (A0)
- no-connect marks 0 -> 2

Commit message: k30p-VME rev.1, MemBird Woodcock rev.1, and frontpanels
Parts:
- U10, U11, U12, U14, U16: value 74ABT16245DL -> 74FCT16245DL
Other:
- moved on the sheet: U10, U11, U12, U14, U16
