File: controllers/bigboy/hardware/BigBoy-Frontpanel/BigBoy-Frontpanel.kicad_pcb (KiCad board)
At the start: 2 copper layers, 19.9 x 128.5 mm, 5 parts

Commit message: k30p-VME rev.1, MemBird Woodcock rev.1, and frontpanels
Parts:
- added ?: , , F.Cu at (82.3, 116.2)
- added ?: , , F.Cu at (81.0, 99.7)
Other:
- outline, holes or cut-outs redrawn
- board text added: "BigBoy"
- board text added: "ETHERNET"
- board text added: "UB1 / UB2"
- board text added: "UL1 / UL2"
- board text added: "UL3 / UL4"
- board text added: "USB"
- board text added: "microSD"
