File: peripherals/membird/hardware/MemBird - Woodcock/Bus.kicad_sch (KiCad schematic)
At the start: 3 parts, among them U2 VME64-P1-3R

Commit message: MemBird - Woodcock Rev.1 Schematic is complete
Connections:
- net ~{SYSCLK}: now reaches U2.a10 (SYSCLK)
- net +5V renamed VBUS
- net ~{VSYSRESET}: no longer names the net of U2.c12 (~{SYSRESET})

Commit message: k30p-VME rev.1, MemBird Woodcock rev.1, and frontpanels
Changed lines of the file:
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@@
 	(bus
 		(pts
-			(xy 27.94 19.05) (xy 43.18 19.05)
+			(xy 31.75 19.05) (xy 43.18 19.05)
 		)
 		(stroke
@@
 	(bus
 		(pts
-			(xy 27.94 15.24) (xy 52.07 15.24)
+			(xy 31.75 15.24) (xy 52.07 15.24)
 		)
 		(stroke
@@
 				)
 				(justify right)
-				(hide yes)
 			)
 		)
@@
 				)
 				(justify right)
-				(hide yes)
 			)
 		)
@@
 				)
 				(justify right)
-				(hide yes)
 			)
 		)
@@
 				)
 				(justify right)
-				(hide yes)
 			)
 		)
@@
 				)
 				(justify right)
-				(hide yes)
 			)
 		)
@@
 				)
 				(justify right)
-				(hide yes)
 			)
 		)
@@
 	(global_label "VD[0..15]"
 		(shape bidirectional)
-		(at 27.94 15.24 180)
-		(fields_autoplaced yes)
-		(effects
-			(font
-				(size 1.27 1.27)
-			)
-			(justify right)
-		)
-		(property "Intersheetrefs" "${INTERSHEET_REFS}"
-			(at 14.9534 15.24 0)
-			(effects
-				(font
-					(size 1.27 1.27)
-				)
-				(justify right)
-				(hide yes)
+		(at 31.75 15.24 180)
+		(fields_autoplaced yes)
+		(effects
+			(font
+				(size 1.27 1.27)
+			)
+			(justify right)
+		)
+		(property "Intersheetrefs" "${INTERSHEET_REFS}"
+			(at 18.7634 15.24 0)
+			(effects
+				(font
+					(size 1.27 1.27)
+				)
+				(justify right)
 			)
 		)
@@
 				)
 				(justify right)
-				(hide yes)
 			)
 		)
@@
 	(global_label "VA[0..23]"
 		(shape input)
-		(at 27.94 19.05 180)
-		(fields_autoplaced yes)
-		(effects
-			(font
-				(size 1.27 1.27)
-			)
-			(justify right)
-		)
-		(property "Intersheetrefs" "${INTERSHEET_REFS}"
-			(at 16.2461 19.05 0)
-			(effects
-				(font
-					(size 1.27 1.27)
-				)
-				(justify right)
-				(hide yes)
+		(at 31.75 19.05 180)
+		(fields_autoplaced yes)
+		(effects
+			(font
+				(size 1.27 1.27)
+			)
+			(justify right)
+		)
+		(property "Intersheetrefs" "${INTERSHEET_REFS}"
+			(at 20.0561 19.05 0)
+			(effects
+				(font
+					(size 1.27 1.27)
+				)
+				(justify right)
 			)
 		)
@@
 				)
 				(justify right)
-				(hide yes)
 			)
 		)
@@
 				)
 				(justify right)
-				(hide yes)
 			)
 		)
@@
 				)
 				(justify right)
-				(hide yes)
 			)
 		)
@@
 				)
 				(justify right)
-				(hide yes)
 			)
 		)
@@
 				)
 				(justify right)
-				(hide yes)
 			)
 		)
@@
 				)
 				(justify right)
-				(hide yes)
 			)
 		)
@@
 				)
 				(justify right)
-				(hide yes)
-			)
-		)
+			)
+		)
